File: KiCad/usb-debug.sch (KiCad schematic (older format))
At the start: 76 parts, among them IC15 TLV70018DCKT, IC16 NCP380HSNAJAAT1G, IC7 HD3SS3220, J11 632723300011, Q1 PMV32UP, T6 BSS138APW

Commit message: Fix DRC errors
Connections:
- net GND: now also R50.1
- net at R50.2: now also IC16.5 (ILIM)
Changed lines of the file:
@@
 	-1   0    0    1
 $EndComp
+Wire Wire Line
+	4400 9750 4400 9700
+Wire Wire Line
+	4400 10100 4400 10050
 $EndSCHEMATC
