File: KiCad/supply.sch (KiCad schematic (older format))
At the start: 74 parts, among them IC10 TPS62823DLCT, IC12 74HC00PW, IC13 SN74LVC1G126DCKR, IC3 TPS54561, IC4 TLV70018DCKT, IC8 LM3671MF-3.3, IC9 LM3671MF-3.3, T3 BSS138APW

Commit message: Added ferrite beads before DC/DC and SOM
Parts:
- removed IC10: TPS62823DLCT, jetson-nano-baseboard-footprints:TPS62823, symbol jetson-nano-baseboard:TPS62823
- removed IC4: TLV70018DCKT, jetson-nano-baseboard-footprints:SC70-5, symbol jetson-nano-baseboard:TLV700
- removed L5: IHLP1212AEERR47M11, jetson-nano-baseboard-footprints:IHLP-1212AE, symbol jetson-nano-baseboard:IHLP1212AEERR47M11
- removed R92: R_0R_0402, jetson-nano-baseboard-footprints:0402-res, symbol jetson-nano-baseboard:R_0R_0402
- added FB1: 742792022, antmicro-footprints:0805-cap, symbol Device:Ferrite_Bead_Small
- added IC10: AP62301Z6-7, antmicro-footprints:SOT-563, symbol antmicroDCDCConverters:AP62301Z6-7
- added IC4: TPS7A0518PDBVT, antmicro-footprints:SOT-23-5, symbol antmicroPMICVoltageRegulatorsLinear:TPS7A0518PDBVT
- added L5: XEL4030-332MEC, antmicro-footprints:Coilcraft-XEL4030, symbol antmicroFixedInductors:XEL4030-332MEC
- C59: value C_2u2_0402 -> C_22u_0603; footprint jetson-nano-baseboard-footprints:0402-cap -> jetson-nano-baseboard-footprints:0603-cap; MPN C1005X5R1A225K050BC -> GRM188R60J226MEA0D; Manufacturer TDK -> MURATA; Val 2u2 -> 22u
- C61: value C_100p_0402 -> C_100n_0402
- R75: value R_0R_0402 -> R_10k_0402
- R76: value R_10k_0402 -> R_0R_0402
- R94: value R_10k_0402 -> R_0R_0402; Val 10k -> 0
Connections:
- wire segments 231 -> 228
Other:
- moved on the sheet: C16, C17, C18, C19, C21, C22, C23, C24, C25, C28, C60, C61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
