File: jetson-nano-baseboard.kicad_sch (KiCad schematic)
At the start: 3 parts

Commit message: Bumped revision to 1.6.1
Other:
- company: (none) -> Antmicro Ltd
Changed lines of the file:
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@@
   (title_block
     (title "Jetson Nano Baseboard")
-    (date "2022-02-04")
-    (rev "1.5.1")
+    (date "2023-04-19")
+    (rev "1.6.1")
+    (company "Antmicro Ltd")
     (comment 1 "www.antmicro.com")
-    (comment 2 "Antmicro Ltd")
   )
   (image (at 77.47 271.6022) (scale 0.15)
