File: supply.kicad_sch (KiCad schematic)
At the start: 98 parts, among them IC12 74HC00PW, IC13 SN74LVC1G126DCKR, IC4 TPS7A0518PDBVT, J12 533980471, T3 BSS138APW, U1 LM3671MF-3.3/NOPB, U2 LM62440-Q1, U3 SN74LXC1T45DBVR, U5 LM3671MF-3.3/NOPB, U6 SIC477ED-T1-GE3

Commit message: Fixed D1 and D9 footprints
Parts:
- removed D1, D9: ESD5B5_0ST1G, jetson-nano-baseboard-footprints:SOD-523, symbol jetson-nano-baseboard:ESD5B5_0ST1G
- added D1, D9: ESD5B5_0ST1G, antmicro-footprints:SOD-523_NP, symbol antmicroTVSDiodes:ESD5B5_0ST1G
Connections:
- net 3V3_SYS: now also D1.2
- net 5V0_SYS: now also D9.2
- net GND: now also D1.1, D9.1
Changed lines of the file:
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@@
+    (pin "2")
+  )
+  (symbol (lib_id "antmicroTVSDiodes:ESD5B5_0ST1G") (at 216.535 67.945 90) (unit 1)
+    (in_bom yes) (on_board yes) (fields_autoplaced)
+    (property "Reference" "D9" (id 0) (at 219.075 66.675 90)
+      (effects (font (size 1.524 1.524)) (justify right))
+    )
+    (property "Value" "ESD5B5_0ST1G" (id 1) (at 219.075 70.485 90)
+      (effects (font (size 1.524 1.524)) (justify right))
+    )
+    (property "Footprint" "antmicro-footprints:SOD-523_NP" (id 2) (at 211.455 62.865 0)
+      (effects (font (size 1.524 1.524)) (justify left) hide)
+    )
+    (property "Datasheet" "https://www.mouser.pl/datasheet/2/308/ESD5B5_0ST1_D-1805066.pdf" (id 3) (at 208.915 62.865 0)
+      (effects (font (size 1.524 1.524)) (justify left) hide)
+    )
+    (property "Manufacturer" "ON Semiconductor" (id 4) (at 188.595 62.865 0)
+      (effects (font (size 1.524 1.524)) (justify left) hide)
+    )
+    (property "MPN" "ESD5B5.0ST1G" (id 5) (at 203.835 62.865 0)
+      (effects (font (size 1.524 1.524)) (justify left) hide)
+    )
+    (pin "1")
+    (pin "2")
+  )
+  (symbol (lib_id "antmicroTVSDiodes:ESD5B5_0ST1G") (at 184.15 152.4 90) (unit 1)
+    (in_bom yes) (on_board yes) (fields_autoplaced)
+    (property "Reference" "D1" (id 0) (at 186.69 151.13 90)
+      (effects (font (size 1.524 1.524)) (justify right))
+    )
+    (property "Value" "ESD5B5_0ST1G" (id 1) (at 186.69 154.94 90)
+      (effects (font (size 1.524 1.524)) (justify right))
+    )
+    (property "Footprint" "antmicro-footprints:SOD-523_NP" (id 2) (at 179.07 147.32 0)
+      (effects (font (size 1.524 1.524)) (justify left) hide)
+    )
+    (property "Datasheet" "https://www.mouser.pl/datasheet/2/308/ESD5B5_0ST1_D-1805066.pdf" (id 3) (at 176.53 147.32 0)
+      (effects (font (size 1.524 1.524)) (justify left) hide)
+    )
+    (property "Manufacturer" "ON Semiconductor" (id 4) (at 156.21 147.32 0)
+      (effects (font (size 1.524 1.524)) (justify left) hide)
+    )
+    (property "MPN" "ESD5B5.0ST1G" (id 5) (at 171.45 147.32 0)
+      (effects (font (size 1.524 1.524)) (justify left) hide)
+    )
+    (pin "1")
     (pin "2")
   )
@@
     )
     (property "MPN" "SMBJ33A" (id 5) (at 240.03 251.46 0)
-      (effects (font (size 1.524 1.524)) (justify left) hide)
-    )
-    (pin "1")
-    (pin "2")
-  )
-  (symbol (lib_id "jetson-nano-baseboard:ESD5B5_0ST1G") (at 216.535 67.945 90) (unit 1)
-    (in_bom yes) (on_board yes) (fields_autoplaced)
-    (property "Reference" "D9" (id 0) (at 219.075 66.675 90)
-      (effects (font (size 1.524 1.524)) (justify right))
-    )
-    (property "Value" "ESD5B5_0ST1G" (id 1) (at 219.075 70.485 90)
-      (effects (font (size 1.524 1.524)) (justify right))
-    )
-    (property "Footprint" "jetson-nano-baseboard-footprints:SOD-523" (id 2) (at 211.455 62.865 0)
-      (effects (font (size 1.524 1.524)) (justify left) hide)
-    )
-    (property "Datasheet" "https://www.mouser.pl/datasheet/2/308/ESD5B5_0ST1_D-1805066.pdf" (id 3) (at 208.915 62.865 0)
-      (effects (font (size 1.524 1.524)) (justify left) hide)
-    )
-    (property "Manufacturer" "ON Semiconductor" (id 4) (at 188.595 62.865 0)
-      (effects (font (size 1.524 1.524)) (justify left) hide)
-    )
-    (property "MPN" "ESD5B5.0ST1G" (id 5) (at 203.835 62.865 0)
       (effects (font (size 1.524 1.524)) (justify left) hide)
     )
@@
     (pin "1")
   )
-  (symbol (lib_id "jetson-nano-baseboard:ESD5B5_0ST1G") (at 184.15 152.4 90) (unit 1)
-    (in_bom yes) (on_board yes) (fields_autoplaced)
-    (property "Reference" "D1" (id 0) (at 186.69 151.13 90)
-      (effects (font (size 1.524 1.524)) (justify right))
-    )
-    (property "Value" "ESD5B5_0ST1G" (id 1) (at 186.69 154.94 90)
-      (effects (font (size 1.524 1.524)) (justify right))
-    )
-    (property "Footprint" "jetson-nano-baseboard-footprints:SOD-523" (id 2) (at 179.07 147.32 0)
-      (effects (font (size 1.524 1.524)) (justify left) hide)
-    )
-    (property "Datasheet" "https://www.mouser.pl/datasheet/2/308/ESD5B5_0ST1_D-1805066.pdf" (id 3) (at 176.53 147.32 0)
-      (effects (font (size 1.524 1.524)) (justify left) hide)
-    )
-    (property "Manufacturer" "ON Semiconductor" (id 4) (at 156.21 147.32 0)
-      (effects (font (size 1.524 1.524)) (justify left) hide)
-    )
-    (property "MPN" "ESD5B5.0ST1G" (id 5) (at 171.45 147.32 0)
-      (effects (font (size 1.524 1.524)) (justify left) hide)
-    )
-    (pin "1")
-    (pin "2")
-  )
   (symbol (lib_id "jetson-nano-baseboard:GND") (at 252.73 261.62 0) (unit 1)

Commit message: Updated loclib and synced it with schematic
Parts:
- D1, D9: footprint antmicro-footprints:SOD-523_NP -> jetson-nano-baseboard-footprints:SOD-523_NP; symbol antmicroTVSDiodes:ESD5B5_0ST1G -> jetson-nano-baseboard:ESD5B5_0ST1G

Commit message: Standardize components
Parts:
- removed F3: 3413_0329_22, jetson-nano-baseboard-footprints:1206, symbol jetson-nano-baseboard:3413_0329_22
- removed U6: SIC477ED-T1-GE3, jetson-nano-baseboard-footprints:SIC47XED-T1-GE3, symbol jetson-nano-baseboard:SIC477ED-T1-GE3
- added F3: F_12A_1206, antmicro-footprints:F_1206_3216Metric, symbol antmicroFuses:F_12A_1206
- added U6: SIC477ED-T1-GE3, antmicro-footprints:SIC47XED-T1-GE3, symbol antmicroDCDCConverters:SIC477ED-T1-GE3
- C16, C18, C60: footprint jetson-nano-baseboard-footprints:0402-cap -> antmicro-footprints:C_0402_1005Metric; symbol jetson-nano-baseboard:C_2u2_0402 -> antmicroCapacitors0402:C_2u2_0402; Author (none) -> Antmicro; License (none) -> Apache-2.0
- C17, C19, C21, C22: footprint jetson-nano-baseboard-footprints:1206-cap -> antmicro-footprints:C_1206_3216Metric; symbol jetson-nano-baseboard:C_10u_1206_50V -> antmicroCapacitorsmisc:C_10u_1206_50V; Author (none) -> Antmicro; License (none) -> Apache-2.0
- C20, C59, C64: footprint jetson-nano-baseboard-footprints:0805-cap -> antmicro-footprints:C_0805_2012Metric; symbol jetson-nano-baseboard:C_47u_0805 -> antmicroCapacitorsmisc:C_47u_0805; Author (none) -> Antmicro; License (none) -> Apache-2.0
- C23, C55, C63, C81: footprint jetson-nano-baseboard-footprints:0603-cap -> antmicro-footprints:C_0603_1608Metric; symbol jetson-nano-baseboard:C_10u_0603 -> antmicroCapacitors0603:C_10u_0603; Author (none) -> Antmicro; License (none) -> Apache-2.0
- C24: footprint jetson-nano-baseboard-footprints:0402-cap -> antmicro-footprints:C_0402_1005Metric; symbol jetson-nano-baseboard:C_6p_0402 -> antmicroCapacitors0402:C_6p_0402; Author (none) -> Antmicro; License (none) -> Apache-2.0; Manufacturer WALSIN -> Walsin
- C25: footprint jetson-nano-baseboard-footprints:0805-cap -> antmicro-footprints:C_0805_2012Metric; symbol jetson-nano-baseboard:C_10u_0805 -> antmicroCapacitorsmisc:C_10u_0805; Author (none) -> Antmicro; License (none) -> Apache-2.0; Manufacturer JOHANSON_DIELECTRICS -> Johanson Technology Inc.
- C28: footprint jetson-nano-baseboard-footprints:0402-res -> antmicro-footprints:C_0402_1005Metric; symbol jetson-nano-baseboard:C_270p_25V_0402 -> antmicroCapacitors0402:C_270p_25V_0402; Author (none) -> Antmicro; License (none) -> Apache-2.0
- C41: footprint jetson-nano-baseboard-footprints:0402-cap -> antmicro-footprints:C_0402_1005Metric; symbol jetson-nano-baseboard:C_47n_0402 -> antmicroCapacitors0402:C_47n_0402; Author (none) -> Antmicro; License (none) -> Apache-2.0; Manufacturer MULTICOMP -> Multicomp
- C56: value C_100n_0402_50V -> C_100n_50V_0402; footprint jetson-nano-baseboard-footprints:0402-cap -> antmicro-footprints:C_0402_1005Metric; symbol jetson-nano-baseboard:C_100n_0402_50V -> antmicroCapacitorsmisc:C_100n_50V_0402; Author (none) -> Antmicro; License (none) -> Apache-2.0
- C57, C71, C83, C86, C88, C89: footprint jetson-nano-baseboard-footprints:0402-cap -> antmicro-footprints:C_0402_1005Metric; symbol jetson-nano-baseboard:C_100n_0402 -> antmicroCapacitors0402:C_100n_0402; Author (none) -> Antmicro; Dielectric (none) -> X5R; License (none) -> Apache-2.0; MPN 0402X104K6R3CT -> GRM155R61H104KE14D; Manufacturer Walsin -> Murata; Voltage (none) -> 50V
- C58: footprint jetson-nano-baseboard-footprints:0402-cap -> antmicro-footprints:C_0402_1005Metric; symbol jetson-nano-baseboard:C_33n_0402 -> antmicroCapacitors0402:C_33n_0402; Author (none) -> Antmicro; License (none) -> Apache-2.0; Manufacturer MULTICOMP -> Multicomp
- C61, C82: footprint jetson-nano-baseboard-footprints:0402-res -> antmicro-footprints:C_0402_1005Metric; symbol jetson-nano-baseboard:C_1n2_50V_0402 -> antmicroCapacitors0402:C_1n2_50V_0402; Author (none) -> Antmicro; License (none) -> Apache-2.0
- C65, C84, C87: footprint jetson-nano-baseboard-footprints:0402-cap -> antmicro-footprints:C_0402_1005Metric; symbol jetson-nano-baseboard:C_1u_0402 -> antmicroCapacitors0402:C_1u_0402; Author (none) -> Antmicro; License (none) -> Apache-2.0
- C85: footprint jetson-nano-baseboard-footprints:0603-cap -> antmicro-footprints:C_0603_1608Metric; symbol jetson-nano-baseboard:C_4u7_0603 -> antmicroCapacitors0603:C_4u7_0603; Author (none) -> Antmicro; License (none) -> Apache-2.0
- D1, D9: footprint jetson-nano-baseboard-footprints:SOD-523_NP -> antmicro-footprints:SOD-523_NP; symbol jetson-nano-baseboard:ESD5B5_0ST1G -> antmicroTVSDiodes:ESD5B5_0ST1G; Author (none) -> Antmicro; License (none) -> Apache-2.0
- D13: footprint jetson-nano-baseboard-footprints:SOD-323 -> antmicro-footprints:D_SOD-323F; symbol jetson-nano-baseboard:diode -> antmicroDiodesRectifiersSingle:1N4148WS; Author (none) -> Antmicro; License (none) -> Apache-2.0
- D14: footprint jetson-nano-baseboard-footprints:D_SMB -> antmicro-footprints:D_SMB; symbol jetson-nano-baseboard:SMBJ33A -> antmicroTVSDiodes:SMBJ33A; Author (none) -> Antmicro; License (none) -> Apache-2.0
- F1, F2: value 04671.25NR -> F_1.25A_0603; footprint jetson-nano-baseboard-footprints:0603-Fuse-Littelfuse-0467 -> antmicro-footprints:F_0603_1608Metric; symbol jetson-nano-baseboard:04671.25NR -> antmicroFuses:F_1.25A_0603; Author (none) -> Antmicro; License (none) -> Apache-2.0; Manufacturer Littelfuse Inc. -> Littelfuse
- FB1: value 74279221100 -> FB_10Z_10A_1206; footprint jetson-nano-baseboard-footprints:1206-res -> antmicro-footprints:FB_1206_3216Metric; symbol jetson-nano-baseboard:74279221100 -> antmicroFerriteBeadsandChips:FB_10Z_10A_1206; Author (none) -> Antmicro; License (none) -> Apache-2.0; Manufacturer Wurth Electronic -> Würth Elektronik
- FB3: value 74279220181 -> FB_180Z_3.1A_0805; footprint jetson-nano-baseboard-footprints:0805-res -> antmicro-footprints:FB_0805_2012Metric; symbol jetson-nano-baseboard:74279220181 -> antmicroFerriteBeadsandChips:FB_180Z_3.1A_0805; Author (none) -> Antmicro; License (none) -> Apache-2.0; Manufacturer Wurth Electronic -> Würth Elektronik
- IC12: value 74HC00PW -> 74HC00_TSSOP; footprint jetson-nano-baseboard-footprints:TSSOP-14 -> antmicro-footprints:TSSOP-14_4.4x5mm_P0.65mm; symbol jetson-nano-baseboard:74HC00PW -> antmicroLogicGatesandInverters:74HC00_TSSOP; Author (none) -> Antmicro; License (none) -> Apache-2.0; MPN 74HC00PW -> 74HC00PW,118; Manufacturer NXP -> Nexperia
- IC13: value SN74LVC1G126DCKR -> SN74LVC1G126_SC-70; footprint jetson-nano-baseboard-footprints:R-PDSO-G5 -> antmicro-footprints:SC-70-5; symbol jetson-nano-baseboard:SN74LVC1G126 -> antmicroLogicGatesandInverters:SN74LVC1G126_SC-70; Author (none) -> Antmicro; License (none) -> Apache-2.0
- IC4: value TPS7A0518PDBVT -> TPS7A0518P_SOT23-5; footprint jetson-nano-baseboard-footprints:SOT-23-5 -> antmicro-footprints:SOT-23-5; symbol jetson-nano-baseboard:TPS7A0518PDBVT -> antmicroPMICVoltageRegulatorsLinear:TPS7A0518P_SOT23-5; Author (none) -> Antmicro; License (none) -> Apache-2.0
- J12: value 533980471 -> PinHeader_PicoBlade_1x4_P1.25mm_SMD; footprint jetson-nano-baseboard-footprints:Molex_PicoBlade_53398-0471_1x04-1MP_P1.25mm_Vertical -> antmicro-footprints:Molex_PicoBlade_53398-0471_1x04-1MP_P1.25mm_Vertical; symbol jetson-nano-baseboard:533980471 -> antmicroRectangularConnectorsHeadersMalePins:PinHeader_PicoBlade_1x4_P1.25mm_SMD; Author (none) -> Antmicro; License (none) -> Apache-2.0
- J4: footprint jetson-nano-baseboard-footprints:DC_SOCKET -> antmicro-footprints:BarrelJack_3167288_Horizontal; symbol jetson-nano-baseboard:DC_SOCKET -> antmicroBarrelAudioConnectors:BarrelJack_3167288; Author (none) -> Antmicro; License (none) -> Apache-2.0
- L1: value XFL4020-222MEC -> L_2u2_3.7A_XFL4020; footprint jetson-nano-baseboard-footprints:XFL4015-122MEC -> antmicro-footprints:L_Coilcraft_XFL4020; symbol jetson-nano-baseboard:XFL4020-222MEC -> antmicroFixedInductors:L_2u2_3.7A_XFL4020; Author (none) -> Antmicro; Imax (none) -> 8.0A; Isat (none) -> 3.7A; License (none) -> Apache-2.0; Size 4.3x4.3 -> 4x4
- L4: footprint jetson-nano-baseboard-footprints:IHLP3232DZ -> antmicro-footprints:L_Vishay_IHLP3232DZ; symbol jetson-nano-baseboard:IHLP3232DZER3R3M01 -> antmicroFixedInductors:IHLP3232DZER3R3M01; Author (none) -> Antmicro; IMax (none) -> 9.2A; ISat (none) -> 20A; License (none) -> Apache-2.0
- L5, L6: value LQH32PN2R2NN0L -> L_2u2_1.6A_1210; footprint jetson-nano-baseboard-footprints:LQH32PN2R2NN0L -> antmicro-footprints:L_1210_3225Metric; symbol jetson-nano-baseboard:LQH32PN2R2NN0L -> antmicroFixedInductors:L_2u2_1.6A_1210; Author (none) -> Antmicro; License (none) -> Apache-2.0; Val (none) -> 2u2/1.6A
- R117: footprint jetson-nano-baseboard-footprints:0402-res -> antmicro-footprints:R_0402_1005Metric; symbol jetson-nano-baseboard:R_52k3_0402 -> antmicroResistors0402:R_52k3_0402; Author (none) -> Antmicro; License (none) -> Apache-2.0; MPN ERJ-2RKF5232X -> CR0402-FX-5232GLF; Manufacturer Panasonic -> Bourns; Tolerance (none) -> 1%
- R118: value R_100k_1%_0402 -> R_100k_0402; footprint jetson-nano-baseboard-footprints:0402 -> antmicro-footprints:R_0402_1005Metric; symbol jetson-nano-baseboard:R_100k_1%_0402 -> antmicroResistors0402:R_100k_0402; Author (none) -> Antmicro; License (none) -> Apache-2.0; MPN ERA-6AEB104V -> CR0402-FX-1003GLF; Manufacturer PANASONIC -> Bourns; Tolerance (none) -> 1%; Val 100k_1% -> 100k
- R119: footprint jetson-nano-baseboard-footprints:0402-res -> antmicro-footprints:R_0402_1005Metric; symbol jetson-nano-baseboard:R_44k2_0402 -> antmicroResistors0402:R_44k2_0402; Author (none) -> Antmicro; License (none) -> Apache-2.0; MPN ERJ2RKF4422X -> CR0402-FX-4422GLF; Manufacturer PANASONIC_ELECTRONIC_COMPONENTS -> Bourns; Tolerance (none) -> 1%
- R120, R39, R44, R46, R52, R95: footprint jetson-nano-baseboard-footprints:0402-res -> antmicro-footprints:R_0402_1005Metric; symbol jetson-nano-baseboard:R_10k_0402 -> antmicroResistors0402:R_10k_0402; Author (none) -> Antmicro; License (none) -> Apache-2.0; MPN CRCW040210K0FKEDHP -> CR0402-FX-1002GLF; Manufacturer VISHAY -> Bourns; Tolerance (none) -> 1%
- R130, R48, R76, R92, R93: footprint jetson-nano-baseboard-footprints:0402-res -> antmicro-footprints:R_0402_1005Metric; symbol jetson-nano-baseboard:R_0R_0402 -> antmicroResistors0402:R_0R_0402; Author (none) -> Antmicro; Current (none) -> 1A; License (none) -> Apache-2.0; Manufacturer PANASONIC -> Panasonic
- R16, R36, R45, R87: footprint jetson-nano-baseboard-footprints:0402-res -> antmicro-footprints:R_0402_1005Metric; symbol jetson-nano-baseboard:R_1k_0402 -> antmicroResistors0402:R_1k_0402; Author (none) -> Antmicro; License (none) -> Apache-2.0; Manufacturer BOURNS -> Bourns; Tolerance (none) -> 1%
- R70: footprint jetson-nano-baseboard-footprints:0402-res -> antmicro-footprints:R_0402_1005Metric; symbol jetson-nano-baseboard:R_100R_0402 -> antmicroResistors0402:R_100R_0402; Author (none) -> Antmicro; License (none) -> Apache-2.0; Manufacturer BOURNS -> Bourns; Tolerance (none) -> 1%
- R74: footprint jetson-nano-baseboard-footprints:0402-res -> antmicro-footprints:R_0402_1005Metric; symbol jetson-nano-baseboard:R_2k_0402 -> antmicroResistors0402:R_2k_0402; Author (none) -> Antmicro; License (none) -> Apache-2.0; MPN CRCW04022K00FKED -> CR0402-FX-2001GLF; Manufacturer VISHAY -> Bourns; Tolerance (none) -> 1%
- R75: footprint jetson-nano-baseboard-footprints:0402-res -> antmicro-footprints:R_0402_1005Metric; symbol jetson-nano-baseboard:R_316k_0402 -> antmicroResistors0402:R_316k_0402; Author (none) -> Antmicro; License (none) -> Apache-2.0; MPN CRCW0402316KFKED -> CR0402-FX-3163GLF; Manufacturer VISHAY -> Bourns; Tolerance (none) -> 1%
- R77: value R_60k4_1%_0402 -> R_60k4_0402; footprint jetson-nano-baseboard-footprints:0402-res -> antmicro-footprints:R_0402_1005Metric; symbol jetson-nano-baseboard:R_60k4_1%_0402 -> antmicroResistors0402:R_60k4_0402; Author (none) -> Antmicro; License (none) -> Apache-2.0; MPN ERJ-2RKF6042X -> CR0402-FX-6042GLF; Manufacturer Panasonic -> Bourns; Tolerance (none) -> 1%; Val 60k4_1% -> 60k4
- R84, R86: footprint jetson-nano-baseboard-footprints:0402-res -> antmicro-footprints:R_0402_1005Metric; symbol jetson-nano-baseboard:R_200k_0402 -> antmicroResistors0402:R_200k_0402; Author (none) -> Antmicro; License (none) -> Apache-2.0; MPN RC0402FR-07200KL -> CR0402-FX-2003GLF; Manufacturer YAGEO_(PHYCOMP) -> Bourns; Tolerance (none) -> 1%
- R85: footprint jetson-nano-baseboard-footprints:0402-res -> antmicro-footprints:R_0402_1005Metric; symbol jetson-nano-baseboard:R_470k_0402 -> antmicroResistors0402:R_470k_0402; Author (none) -> Antmicro; License (none) -> Apache-2.0; MPN RC0402FR-07470KL -> CR0402-FX-4703GLF; Manufacturer YAGEO -> Bourns; Tolerance (none) -> 1%
- R89: footprint jetson-nano-baseboard-footprints:0402-res -> antmicro-footprints:R_0402_1005Metric; symbol jetson-nano-baseboard:R_3R3_0402 -> antmicroResistors0402:R_3R3_0402; Author (none) -> Antmicro; License (none) -> Apache-2.0; MPN ERJ2GEJ3R3X -> CR0402-FX-3R30GLF; Manufacturer Panasonic -> Bourns; Tolerance (none) -> 1%
- R90: footprint jetson-nano-baseboard-footprints:0402-res -> antmicro-footprints:R_0402_1005Metric; symbol jetson-nano-baseboard:R_26k7_0402 -> antmicroResistors0402:R_26k7_0402; Author (none) -> Antmicro; License (none) -> Apache-2.0; MPN MCMR04X2672FTL -> CR0402-FX-2672GLF; Manufacturer Multicomp -> Bourns; Tolerance (none) -> 1%
- R91, R96: footprint jetson-nano-baseboard-footprints:0402-res -> antmicro-footprints:R_0402_1005Metric; symbol jetson-nano-baseboard:R_100k_0402 -> antmicroResistors0402:R_100k_0402; Author (none) -> Antmicro; License (none) -> Apache-2.0; MPN CRCW0402100KFKEDHP -> CR0402-FX-1003GLF; Manufacturer VISHAY -> Bourns; Tolerance (none) -> 1%
- R94: value R_8k66_1%_0402 -> R_8k66_0402; footprint jetson-nano-baseboard-footprints:0402-res -> antmicro-footprints:R_0402_1005Metric; symbol jetson-nano-baseboard:R_8k66_1%_0402 -> antmicroResistors0402:R_8k66_0402; Author (none) -> Antmicro; License (none) -> Apache-2.0; MPN RC0402FR-078K66L -> CR0402-FX-8661GLF; Manufacturer YAGEO -> Bourns; Tolerance (none) -> 1%; Val 8k66_1% -> 8k66
- T3: value BSS138APW -> BSS138PW; footprint jetson-nano-baseboard-footprints:SC70-3 -> antmicro-footprints:SC70-3; symbol jetson-nano-baseboard:BSS138APW -> antmicroTransistorsFETsMOSFETsSingle:BSS138PW; Author (none) -> Antmicro; License (none) -> Apache-2.0; Manufacturer ON Semiconductor -> Nexperia
- TP11, TP12, TP15, TP40, TP41: value Testpad -> TP_1.5mm_SMD; footprint jetson-nano-baseboard-footprints:TP-R-1.5 -> antmicro-footprints:TP_SMD_1.5mm; symbol jetson-nano-baseboard:Testpad -> antmicroTestPoints:TP_1.5mm_SMD; Author (none) -> Antmicro; License (none) -> Apache-2.0
- TP16, TP17, TP42, TP44, TP47, TP5, TP8: value ~ -> TP_1.5mm_SMD; footprint jetson-nano-baseboard-footprints:TP-R-1.5 -> antmicro-footprints:TP_SMD_1.5mm; symbol jetson-nano-baseboard:Testpad -> antmicroTestPoints:TP_1.5mm_SMD; Author (none) -> Antmicro; License (none) -> Apache-2.0
- U1, U5: value LM3671MF-3.3/NOPB -> LM3671MF-3.3_SOT; footprint jetson-nano-baseboard-footprints:SOT-23-5 -> antmicro-footprints:SOT-23-5; symbol jetson-nano-baseboard:LM3671MF-3.3_NOPB -> antmicroPMICVoltageRegulatorsDCDCSwitchingRegulators:LM3671MF-3.3_SOT; Author (none) -> Antmicro; License (none) -> Apache-2.0
- U2: footprint jetson-nano-baseboard-footprints:VQFN-14-HR -> antmicro-footprints:VQFN-14-HR; symbol jetson-nano-baseboard:LM62440-Q1 -> antmicroDCDCConverters:LM62440-Q1; Author (none) -> Antmicro; License (none) -> Apache-2.0
- U3: footprint jetson-nano-baseboard-footprints:SOT-23-6 -> antmicro-footprints:SOT-23-6; symbol jetson-nano-baseboard:SN74LXC1T45DBVR -> antmicroLogicTranslatorsLevelShifters:SN74LXC1T45DBVR; Author (none) -> Antmicro; License (none) -> Apache-2.0
Connections:
- net #RESET: now also R39.1, R44.1, R52.1, R92.1; no longer R39.2, R44.2, R52.2, R92.2
- net #SHUTDOWN_REQ: now also R86.2; no longer R86.1
- net 1V8_SYS: now also C86.1; no longer C86.2
- net 3V3_EN: now also R44.2; no longer R44.1
- net 3V3_FFC2: now also F2.2; no longer F2.1
- net 3V3_SW: now also L1.1; no longer L1.2
- net 3V3_SYS: now also L1.2; no longer L1.1
- net 5V0_SYS: now also C71.1, C82.2, C83.1, C88.1, R46.1, R84.1, R86.1, R93.2; no longer C71.2, C82.1, C83.2, C88.2, R46.2, R84.2, R86.2, R93.1
- net 5V_BOOT: now also C57.2, U6.4 (BOOT); no longer C57.1
- net 5V_COMP: now also U6.21 (COMP)
- net 5V_EN: now also U6.3 (EN)
- net 5V_FB: now also U6.22 (V_{FB})
- net 5V_FSW: now also U6.24 (f_{SW})
- net 5V_ILIM: now also R76.2, U6.25 (I_{LIMIT}); no longer R76.1
- net 5V_MODE: now also U6.27 (MODE)
- net 5V_PHASE: now also U6.5 (PHASE), U6.6 (PHASE)
- net 5V_SNS: now also C61.2, C82.1; no longer C61.1, C82.2
- net 5V_SS: now also U6.19 (SS)
- net 5V_SW: now also U6.12 (SW), U6.13 (SW), U6.14 (SW)
- net 5V_VIN: now also U6.1 (V_{CIN}), U6.7 (V_{IN}), U6.8 (V_{IN})
- net FAN_TACH_5V: now also R46.2; no longer R46.1
- net GND: now also C28.2, C41.2, C63.2, C71.2, C83.2, C86.2, C88.2, U6.10 (PGND), U6.11 (PGND), U6.17 (PGND), U6.23 (AGND), U6.28 (AGND), U6.9 (PGND); no longer C28.1, C41.1, C63.1, C71.1, C83.1, C86.1, C88.1
- net PWR_GOOD: now also R96.1, U6.2 (P_{GOOD}); no longer R96.2
- net Q: now also D13.K; no longer D13.C
- net QDEL: now also C63.1; no longer C63.2
- net VDD_5V_DCDC: now also R76.1, R96.2, U6.26 (V_{DD}); no longer R76.2, R96.1
- net VDRV_5V_DCDC: now also U6.16 (V_{DRV})
- net VIN: now also F3.2
- net \~{PWR_SET}: now also C41.1, R84.2; no longer C41.2, R84.1
- net at J4.1: now also F3.1
- net at IC4.3 (EN): now also R92.2; no longer R92.1
- net at C55.1, L6.2, TP8.1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: now also F2.1; no longer F2.2
- net at R89.1: now also C57.1; no longer C57.2
- net at U1.3 (EN): now also R39.2; no longer R39.1
- net at U5.3 (EN): now also R52.2; no longer R52.1
- net at R75.2: now also C28.1; no longer C28.2
- new net: C61.1, R93.1, U6.20 (V_{SNS})
- no-connect marks 3 -> 5
Other:
- moved on the sheet: C16, C17, C18, C19, C20, C21, C22, C23, C24, C25, C28, C41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

Commit message: [#56834] Fix components links
Parts:
- C16, C18, C60: footprint antmicro-footprints:C_0402_1005Metric -> jetson-nano-baseboard-footprints:C_0402_1005Metric; symbol antmicroCapacitors0402:C_2u2_0402 -> jetson-nano-baseboard:C_2u2_0402
- C17, C19, C21, C22: footprint antmicro-footprints:C_1206_3216Metric -> jetson-nano-baseboard-footprints:C_1206_3216Metric; symbol antmicroCapacitorsmisc:C_10u_1206_50V -> jetson-nano-baseboard:C_10u_1206_50V; Val 10u/50V -> 10u; Voltage (none) -> 50V
- C20, C59, C64: footprint antmicro-footprints:C_0805_2012Metric -> jetson-nano-baseboard-footprints:C_0805_2012Metric; symbol antmicroCapacitorsmisc:C_47u_0805 -> jetson-nano-baseboard:C_47u_0805
- C23, C55, C63, C81: footprint antmicro-footprints:C_0603_1608Metric -> jetson-nano-baseboard-footprints:C_0603_1608Metric; symbol antmicroCapacitors0603:C_10u_0603 -> jetson-nano-baseboard:C_10u_0603
- C24: footprint antmicro-footprints:C_0402_1005Metric -> jetson-nano-baseboard-footprints:C_0402_1005Metric; symbol antmicroCapacitors0402:C_6p_0402 -> jetson-nano-baseboard:C_6p_0402; now not fitted; now left out of the parts list
- C25: footprint antmicro-footprints:C_0805_2012Metric -> jetson-nano-baseboard-footprints:C_0805_2012Metric; symbol antmicroCapacitorsmisc:C_10u_0805 -> jetson-nano-baseboard:C_10u_0805; Manufacturer Johanson Technology Inc. -> Johanson Technology
- C28: footprint antmicro-footprints:C_0402_1005Metric -> jetson-nano-baseboard-footprints:C_0402_1005Metric; symbol antmicroCapacitors0402:C_270p_25V_0402 -> jetson-nano-baseboard:C_270p_25V_0402; Val 270p_25V -> 270p; Voltage (none) -> 25V; now not fitted; now left out of the parts list
- C41: footprint antmicro-footprints:C_0402_1005Metric -> jetson-nano-baseboard-footprints:C_0402_1005Metric; symbol antmicroCapacitors0402:C_47n_0402 -> jetson-nano-baseboard:C_47n_0402; MPN MC0402X473K160CT -> GRM155R61H474KE11D; Manufacturer Multicomp -> Murata
- C56: footprint antmicro-footprints:C_0402_1005Metric -> jetson-nano-baseboard-footprints:C_0402_1005Metric; symbol antmicroCapacitorsmisc:C_100n_50V_0402 -> jetson-nano-baseboard:C_100n_50V_0402; Val 100n/50V -> 100n; Voltage (none) -> 50V
- C57, C71, C83, C86, C88, C89: footprint antmicro-footprints:C_0402_1005Metric -> jetson-nano-baseboard-footprints:C_0402_1005Metric; symbol antmicroCapacitors0402:C_100n_0402 -> jetson-nano-baseboard:C_100n_0402
- C58: footprint antmicro-footprints:C_0402_1005Metric -> jetson-nano-baseboard-footprints:C_0402_1005Metric; symbol antmicroCapacitors0402:C_33n_0402 -> jetson-nano-baseboard:C_33n_0402; MPN MC0402B333K250CT -> GCM155R71E333KA55D; Manufacturer Multicomp -> Murata
- C61, C82: footprint antmicro-footprints:C_0402_1005Metric -> jetson-nano-baseboard-footprints:C_0402_1005Metric; symbol antmicroCapacitors0402:C_1n2_50V_0402 -> jetson-nano-baseboard:C_1n2_50V_0402; Val 1n2_50V -> 1n2; Voltage (none) -> 50V; now not fitted; now left out of the parts list
- C65, C84, C87: footprint antmicro-footprints:C_0402_1005Metric -> jetson-nano-baseboard-footprints:C_0402_1005Metric; symbol antmicroCapacitors0402:C_1u_0402 -> jetson-nano-baseboard:C_1u_0402
- C85: footprint antmicro-footprints:C_0603_1608Metric -> jetson-nano-baseboard-footprints:C_0603_1608Metric; symbol antmicroCapacitors0603:C_4u7_0603 -> jetson-nano-baseboard:C_4u7_0603
- D1, D9: footprint antmicro-footprints:SOD-523_NP -> jetson-nano-baseboard-footprints:SOD-523_NP; symbol antmicroTVSDiodes:ESD5B5_0ST1G -> jetson-nano-baseboard:ESD5B5_0ST1G
- D13: footprint antmicro-footprints:D_SOD-323F -> jetson-nano-baseboard-footprints:D_SOD-323F; symbol antmicroDiodesRectifiersSingle:1N4148WS -> jetson-nano-baseboard:1N4148WS
- D14: footprint antmicro-footprints:D_SMB -> jetson-nano-baseboard-footprints:D_SMB; symbol antmicroTVSDiodes:SMBJ33A -> jetson-nano-baseboard:SMBJ33A
- F1, F2: footprint antmicro-footprints:F_0603_1608Metric -> jetson-nano-baseboard-footprints:F_0603_1608Metric; symbol antmicroFuses:F_1.25A_0603 -> jetson-nano-baseboard:F_1.25A_0603
- F3: footprint antmicro-footprints:F_1206_3216Metric -> jetson-nano-baseboard-footprints:F_1206_3216Metric; symbol antmicroFuses:F_12A_1206 -> jetson-nano-baseboard:F_12A_1206
- FB1: value FB_10Z_10A_1206 -> FB_10Z_10A_WE-MPSB_1206; footprint antmicro-footprints:FB_1206_3216Metric -> jetson-nano-baseboard-footprints:FB_1206_3216Metric; symbol antmicroFerriteBeadsandChips:FB_10Z_10A_1206 -> jetson-nano-baseboard:FB_10Z_10A_WE-MPSB_1206
- FB3: value FB_180Z_3.1A_0805 -> FB_180Z_3.1A_WE-MPSB_0805; footprint antmicro-footprints:FB_0805_2012Metric -> jetson-nano-baseboard-footprints:FB_0805_2012Metric; symbol antmicroFerriteBeadsandChips:FB_180Z_3.1A_0805 -> jetson-nano-baseboard:FB_180Z_3.1A_WE-MPSB_0805
- IC12: footprint antmicro-footprints:TSSOP-14_4.4x5mm_P0.65mm -> jetson-nano-baseboard-footprints:TSSOP-14_4.4x5mm_P0.65mm; symbol antmicroLogicGatesandInverters:74HC00_TSSOP -> jetson-nano-baseboard:74HC00_TSSOP
- IC13: footprint antmicro-footprints:SC-70-5 -> jetson-nano-baseboard-footprints:SC-70-5; symbol antmicroLogicGatesandInverters:SN74LVC1G126_SC-70 -> jetson-nano-baseboard:SN74LVC1G126_SC-70
- IC4: footprint antmicro-footprints:SOT-23-5 -> jetson-nano-baseboard-footprints:SOT-23-5; symbol antmicroPMICVoltageRegulatorsLinear:TPS7A0518P_SOT23-5 -> jetson-nano-baseboard:TPS7A0518P_SOT23-5
- J12: value PinHeader_PicoBlade_1x4_P1.25mm_SMD -> Molex_PicoBlade_1x4_0533980471; footprint antmicro-footprints:Molex_PicoBlade_53398-0471_1x04-1MP_P1.25mm_Vertical -> jetson-nano-baseboard-footprints:Conn_Molex_PicoBlade_1x4_0533980471; symbol antmicroRectangularConnectorsHeadersMalePins:PinHeader_PicoBlade_1x4_P1.25mm_SMD -> jetson-nano-baseboard:Molex_PicoBlade_1x4_0533980471
- J4: value ~ -> BarrelJack_Pin2mm_MJ-179PH; footprint antmicro-footprints:BarrelJack_3167288_Horizontal -> jetson-nano-baseboard-footprints:BarrelJack_Pin2mm_MJ-179PH; symbol antmicroBarrelAudioConnectors:BarrelJack_3167288 -> jetson-nano-baseboard:BarrelJack_Pin2mm_MJ-179PH; Manufacturer Multicomp -> Multicomp Pro
- L1: value L_2u2_3.7A_XFL4020 -> L_2u2_8A_Coilcraft-XFL4020; footprint antmicro-footprints:L_Coilcraft_XFL4020 -> jetson-nano-baseboard-footprints:L_Coilcraft-XFL4020; symbol antmicroFixedInductors:L_2u2_3.7A_XFL4020 -> jetson-nano-baseboard:L_2u2_8A_Coilcraft-XFL4020; Imax 8.0A -> 8A; Size 4x4 -> 4.0x4.0; Val 2u2/3.7A -> 2u2/8A
- L4: value IHLP3232DZER3R3M01 -> L_3u3_9.2A_Vishay-IHLP-3232DZ-01; footprint antmicro-footprints:L_Vishay_IHLP3232DZ -> jetson-nano-baseboard-footprints:L_Vishay-IHLP3232DZ; symbol antmicroFixedInductors:IHLP3232DZER3R3M01 -> jetson-nano-baseboard:L_3u3_9.2A_Vishay-IHLP-3232DZ-01; IMax 9.2A -> 9.2 A; ISat 20A -> 20 A
- L5, L6: footprint antmicro-footprints:L_1210_3225Metric -> jetson-nano-baseboard-footprints:L_1210_3225Metric; symbol antmicroFixedInductors:L_2u2_1.6A_1210 -> jetson-nano-baseboard:L_2u2_1.6A_1210; IMax (none) -> 1.6 A; Size (none) -> 3.2x2.5
- R117: footprint antmicro-footprints:R_0402_1005Metric -> jetson-nano-baseboard-footprints:R_0402_1005Metric; symbol antmicroResistors0402:R_52k3_0402 -> jetson-nano-baseboard:R_52k3_0402
- R118: footprint antmicro-footprints:R_0402_1005Metric -> jetson-nano-baseboard-footprints:R_0402_1005Metric; symbol antmicroResistors0402:R_100k_0402 -> jetson-nano-baseboard:R_100k_0402; now not fitted; now left out of the parts list
- R119: footprint antmicro-footprints:R_0402_1005Metric -> jetson-nano-baseboard-footprints:R_0402_1005Metric; symbol antmicroResistors0402:R_44k2_0402 -> jetson-nano-baseboard:R_44k2_0402; now not fitted; now left out of the parts list
- R120, R39, R44, R46, R52, R95: footprint antmicro-footprints:R_0402_1005Metric -> jetson-nano-baseboard-footprints:R_0402_1005Metric; symbol antmicroResistors0402:R_10k_0402 -> jetson-nano-baseboard:R_10k_0402
- R130: footprint antmicro-footprints:R_0402_1005Metric -> jetson-nano-baseboard-footprints:R_0402_1005Metric; symbol antmicroResistors0402:R_0R_0402 -> jetson-nano-baseboard:R_0R_0402; now not fitted; now left out of the parts list
- R16, R36: footprint antmicro-footprints:R_0402_1005Metric -> jetson-nano-baseboard-footprints:R_0402_1005Metric; symbol antmicroResistors0402:R_1k_0402 -> jetson-nano-baseboard:R_1k_0402
- R45, R87: footprint antmicro-footprints:R_0402_1005Metric -> jetson-nano-baseboard-footprints:R_0402_1005Metric; symbol antmicroResistors0402:R_1k_0402 -> jetson-nano-baseboard:R_1k_0402; now not fitted; now left out of the parts list
- R48, R76, R92, R93: footprint antmicro-footprints:R_0402_1005Metric -> jetson-nano-baseboard-footprints:R_0402_1005Metric; symbol antmicroResistors0402:R_0R_0402 -> jetson-nano-baseboard:R_0R_0402
- R70: footprint antmicro-footprints:R_0402_1005Metric -> jetson-nano-baseboard-footprints:R_0402_1005Metric; symbol antmicroResistors0402:R_100R_0402 -> jetson-nano-baseboard:R_100R_0402
- R74: footprint antmicro-footprints:R_0402_1005Metric -> jetson-nano-baseboard-footprints:R_0402_1005Metric; symbol antmicroResistors0402:R_2k_0402 -> jetson-nano-baseboard:R_2k_0402
- R75: footprint antmicro-footprints:R_0402_1005Metric -> jetson-nano-baseboard-footprints:R_0402_1005Metric; symbol antmicroResistors0402:R_316k_0402 -> jetson-nano-baseboard:R_316k_0402; now not fitted; now left out of the parts list
- R77: footprint antmicro-footprints:R_0402_1005Metric -> jetson-nano-baseboard-footprints:R_0402_1005Metric; symbol antmicroResistors0402:R_60k4_0402 -> jetson-nano-baseboard:R_60k4_0402; now not fitted; now left out of the parts list
- R84, R86: footprint antmicro-footprints:R_0402_1005Metric -> jetson-nano-baseboard-footprints:R_0402_1005Metric; symbol antmicroResistors0402:R_200k_0402 -> jetson-nano-baseboard:R_200k_0402
- R85: footprint antmicro-footprints:R_0402_1005Metric -> jetson-nano-baseboard-footprints:R_0402_1005Metric; symbol antmicroResistors0402:R_470k_0402 -> jetson-nano-baseboard:R_470k_0402
- R89: footprint antmicro-footprints:R_0402_1005Metric -> jetson-nano-baseboard-footprints:R_0402_1005Metric; symbol antmicroResistors0402:R_3R3_0402 -> jetson-nano-baseboard:R_3R3_0402
- R90: footprint antmicro-footprints:R_0402_1005Metric -> jetson-nano-baseboard-footprints:R_0402_1005Metric; symbol antmicroResistors0402:R_26k7_0402 -> jetson-nano-baseboard:R_26k7_0402
- R91, R96: footprint antmicro-footprints:R_0402_1005Metric -> jetson-nano-baseboard-footprints:R_0402_1005Metric; symbol antmicroResistors0402:R_100k_0402 -> jetson-nano-baseboard:R_100k_0402
- R94: footprint antmicro-footprints:R_0402_1005Metric -> jetson-nano-baseboard-footprints:R_0402_1005Metric; symbol antmicroResistors0402:R_8k66_0402 -> jetson-nano-baseboard:R_8k66_0402; now not fitted; now left out of the parts list
- T3: footprint antmicro-footprints:SC70-3 -> jetson-nano-baseboard-footprints:SC70-3; symbol antmicroTransistorsFETsMOSFETsSingle:BSS138PW -> jetson-nano-baseboard:BSS138PW
- TP11, TP12, TP15, TP16, TP17, TP40, TP41, TP42, TP44, TP47, TP5, TP8: footprint antmicro-footprints:TP_SMD_1.5mm -> jetson-nano-baseboard-footprints:TP_SMD_1.5mm; symbol antmicroTestPoints:TP_1.5mm_SMD -> jetson-nano-baseboard:TP_1.5mm_SMD; MPN N/A -> (none); Manufacturer N/A -> (none)
- U1, U5: footprint antmicro-footprints:SOT-23-5 -> jetson-nano-baseboard-footprints:SOT-23-5; symbol antmicroPMICVoltageRegulatorsDCDCSwitchingRegulators:LM3671MF-3.3_SOT -> jetson-nano-baseboard:LM3671MF-3.3_SOT
- U2: footprint antmicro-footprints:VQFN-14-HR -> jetson-nano-baseboard-footprints:VQFN-HR-14_3.5x4mm; symbol antmicroDCDCConverters:LM62440-Q1 -> jetson-nano-baseboard:LM62440-Q1
- U3: footprint antmicro-footprints:SOT-23-6 -> jetson-nano-baseboard-footprints:SOT-23-6; symbol antmicroLogicTranslatorsLevelShifters:SN74LXC1T45DBVR -> jetson-nano-baseboard:SN74LXC1T45DBVR
- U6: footprint antmicro-footprints:SIC47XED-T1-GE3 -> jetson-nano-baseboard-footprints:SIC47XED-T1-GE3; symbol antmicroDCDCConverters:SIC477ED-T1-GE3 -> jetson-nano-baseboard:SIC477ED-T1-GE3
