File: supply.kicad_sch (KiCad schematic)
At the start: 98 parts, among them IC12 74HC00_TSSOP, IC13 SN74LVC1G126_SC-70, IC4 TPS7A0518P_SOT23-5, J12 Molex_PicoBlade_1x4_0533980471, J4 BarrelJack_Pin2mm_MJ-179PH, T3 BSS138PW, U1 LM3671MF-3.3_SOT, U2 LM62440-Q1, U3 SN74LXC1T45DBVR, U5 LM3671MF-3.3_SOT, U6 SIC477ED-T1-GE3

Commit message: [#57913] fix 2309413-1
Parts:
- C16, C18, C60: footprint jetson-nano-baseboard-footprints:C_0402_1005Metric -> antmicro-footprints:C_0402_1005Metric; symbol jetson-nano-baseboard:C_2u2_0402 -> antmicroCapacitors0402:C_2u2_0402
- C17, C19, C21, C22: footprint jetson-nano-baseboard-footprints:C_1206_3216Metric -> antmicro-footprints:C_1206_3216Metric; symbol jetson-nano-baseboard:C_10u_1206_50V -> antmicroCapacitorsmisc:C_10u_1206_50V
- C20, C59, C64: footprint jetson-nano-baseboard-footprints:C_0805_2012Metric -> antmicro-footprints:C_0805_2012Metric; symbol jetson-nano-baseboard:C_47u_0805 -> antmicroCapacitorsmisc:C_47u_0805
- C23, C55, C63, C81: footprint jetson-nano-baseboard-footprints:C_0603_1608Metric -> antmicro-footprints:C_0603_1608Metric; symbol jetson-nano-baseboard:C_10u_0603 -> antmicroCapacitors0603:C_10u_0603
- C24: footprint jetson-nano-baseboard-footprints:C_0402_1005Metric -> antmicro-footprints:C_0402_1005Metric; symbol jetson-nano-baseboard:C_6p_0402 -> antmicroCapacitors0402:C_6p_0402
- C25: footprint jetson-nano-baseboard-footprints:C_0805_2012Metric -> antmicro-footprints:C_0805_2012Metric; symbol jetson-nano-baseboard:C_10u_0805 -> antmicroCapacitorsmisc:C_10u_0805
- C28: footprint jetson-nano-baseboard-footprints:C_0402_1005Metric -> antmicro-footprints:C_0402_1005Metric; symbol jetson-nano-baseboard:C_270p_25V_0402 -> antmicroCapacitors0402:C_270p_25V_0402
- C41: footprint jetson-nano-baseboard-footprints:C_0402_1005Metric -> antmicro-footprints:C_0402_1005Metric; symbol jetson-nano-baseboard:C_47n_0402 -> antmicroCapacitors0402:C_47n_0402
- C56: footprint jetson-nano-baseboard-footprints:C_0402_1005Metric -> antmicro-footprints:C_0402_1005Metric; symbol jetson-nano-baseboard:C_100n_50V_0402 -> antmicroCapacitorsmisc:C_100n_50V_0402
- C57, C71, C83, C86, C88, C89: footprint jetson-nano-baseboard-footprints:C_0402_1005Metric -> antmicro-footprints:C_0402_1005Metric; symbol jetson-nano-baseboard:C_100n_0402 -> antmicroCapacitors0402:C_100n_0402
- C58: footprint jetson-nano-baseboard-footprints:C_0402_1005Metric -> antmicro-footprints:C_0402_1005Metric; symbol jetson-nano-baseboard:C_33n_0402 -> antmicroCapacitors0402:C_33n_0402
- C61, C82: footprint jetson-nano-baseboard-footprints:C_0402_1005Metric -> antmicro-footprints:C_0402_1005Metric; symbol jetson-nano-baseboard:C_1n2_50V_0402 -> antmicroCapacitors0402:C_1n2_50V_0402
- C65, C84, C87: footprint jetson-nano-baseboard-footprints:C_0402_1005Metric -> antmicro-footprints:C_0402_1005Metric; symbol jetson-nano-baseboard:C_1u_0402 -> antmicroCapacitors0402:C_1u_0402
- C85: footprint jetson-nano-baseboard-footprints:C_0603_1608Metric -> antmicro-footprints:C_0603_1608Metric; symbol jetson-nano-baseboard:C_4u7_0603 -> antmicroCapacitors0603:C_4u7_0603
- D1, D9: footprint jetson-nano-baseboard-footprints:SOD-523_NP -> antmicro-footprints:SOD-523_NP; symbol jetson-nano-baseboard:ESD5B5_0ST1G -> antmicroTVSDiodes:ESD5B5_0ST1G
- D13: footprint jetson-nano-baseboard-footprints:D_SOD-323F -> antmicro-footprints:D_SOD-323F; symbol jetson-nano-baseboard:1N4148WS -> antmicroDiodesRectifiersSingle:1N4148WS
- D14: footprint jetson-nano-baseboard-footprints:D_SMB -> antmicro-footprints:D_SMB; symbol jetson-nano-baseboard:SMBJ33A -> antmicroTVSDiodes:SMBJ33A
- F1, F2: footprint jetson-nano-baseboard-footprints:F_0603_1608Metric -> antmicro-footprints:F_0603_1608Metric; symbol jetson-nano-baseboard:F_1.25A_0603 -> antmicroFuses:F_1.25A_0603
- F3: footprint jetson-nano-baseboard-footprints:F_1206_3216Metric -> antmicro-footprints:F_1206_3216Metric; symbol jetson-nano-baseboard:F_12A_1206 -> antmicroFuses:F_12A_1206
- FB1: footprint jetson-nano-baseboard-footprints:FB_1206_3216Metric -> antmicro-footprints:FB_1206_3216Metric; symbol jetson-nano-baseboard:FB_10Z_10A_WE-MPSB_1206 -> antmicroFerriteBeadsandChips:FB_10Z_10A_WE-MPSB_1206
- FB3: footprint jetson-nano-baseboard-footprints:FB_0805_2012Metric -> antmicro-footprints:FB_0805_2012Metric; symbol jetson-nano-baseboard:FB_180Z_3.1A_WE-MPSB_0805 -> antmicroFerriteBeadsandChips:FB_180Z_3.1A_WE-MPSB_0805
- IC12: footprint jetson-nano-baseboard-footprints:TSSOP-14_4.4x5mm_P0.65mm -> antmicro-footprints:TSSOP-14_4.4x5mm_P0.65mm; symbol jetson-nano-baseboard:74HC00_TSSOP -> antmicroLogicGatesandInverters:74HC00_TSSOP
- IC13: footprint jetson-nano-baseboard-footprints:SC-70-5 -> antmicro-footprints:SC-70-5; symbol jetson-nano-baseboard:SN74LVC1G126_SC-70 -> antmicroLogicGatesandInverters:SN74LVC1G126_SC-70
- IC4: footprint jetson-nano-baseboard-footprints:SOT-23-5 -> antmicro-footprints:SOT-23-5; symbol jetson-nano-baseboard:TPS7A0518P_SOT23-5 -> antmicroPMICVoltageRegulatorsLinear:TPS7A0518P_SOT23-5
- J12: footprint jetson-nano-baseboard-footprints:Conn_Molex_PicoBlade_1x4_0533980471 -> antmicro-footprints:Conn_Molex_PicoBlade_1x4_0533980471; symbol jetson-nano-baseboard:Molex_PicoBlade_1x4_0533980471 -> antmicroWire2BoardConnectors:Molex_PicoBlade_1x4_0533980471
- J4: footprint jetson-nano-baseboard-footprints:BarrelJack_Pin2mm_MJ-179PH -> antmicro-footprints:BarrelJack_Pin2mm_MJ-179PH; symbol jetson-nano-baseboard:BarrelJack_Pin2mm_MJ-179PH -> antmicroBarrelPowerConnectors:BarrelJack_Pin2mm_MJ-179PH
- L1: footprint jetson-nano-baseboard-footprints:L_Coilcraft-XFL4020 -> antmicro-footprints:L_Coilcraft-XFL4020; symbol jetson-nano-baseboard:L_2u2_8A_Coilcraft-XFL4020 -> antmicroFixedInductors:L_2u2_8A_Coilcraft-XFL4020
- L4: footprint jetson-nano-baseboard-footprints:L_Vishay-IHLP3232DZ -> antmicro-footprints:L_Vishay-IHLP3232DZ; symbol jetson-nano-baseboard:L_3u3_9.2A_Vishay-IHLP-3232DZ-01 -> antmicroFixedInductors:L_3u3_9.2A_Vishay-IHLP-3232DZ-01
- L5, L6: footprint jetson-nano-baseboard-footprints:L_1210_3225Metric -> antmicro-footprints:L_1210_3225Metric; symbol jetson-nano-baseboard:L_2u2_1.6A_1210 -> antmicroFixedInductors:L_2u2_1.6A_1210
- R117: footprint jetson-nano-baseboard-footprints:R_0402_1005Metric -> antmicro-footprints:R_0402_1005Metric; symbol jetson-nano-baseboard:R_52k3_0402 -> antmicroResistors0402:R_52k3_0402
- R118, R91, R96: footprint jetson-nano-baseboard-footprints:R_0402_1005Metric -> antmicro-footprints:R_0402_1005Metric; symbol jetson-nano-baseboard:R_100k_0402 -> antmicroResistors0402:R_100k_0402
- R119: footprint jetson-nano-baseboard-footprints:R_0402_1005Metric -> antmicro-footprints:R_0402_1005Metric; symbol jetson-nano-baseboard:R_44k2_0402 -> antmicroResistors0402:R_44k2_0402
- R120, R39, R44, R46, R52, R95: footprint jetson-nano-baseboard-footprints:R_0402_1005Metric -> antmicro-footprints:R_0402_1005Metric; symbol jetson-nano-baseboard:R_10k_0402 -> antmicroResistors0402:R_10k_0402
- R130, R48, R76, R92, R93: footprint jetson-nano-baseboard-footprints:R_0402_1005Metric -> antmicro-footprints:R_0402_1005Metric; symbol jetson-nano-baseboard:R_0R_0402 -> antmicroResistors0402:R_0R_0402
- R16, R36, R45, R87: footprint jetson-nano-baseboard-footprints:R_0402_1005Metric -> antmicro-footprints:R_0402_1005Metric; symbol jetson-nano-baseboard:R_1k_0402 -> antmicroResistors0402:R_1k_0402
- R70: footprint jetson-nano-baseboard-footprints:R_0402_1005Metric -> antmicro-footprints:R_0402_1005Metric; symbol jetson-nano-baseboard:R_100R_0402 -> antmicroResistors0402:R_100R_0402
- R74: footprint jetson-nano-baseboard-footprints:R_0402_1005Metric -> antmicro-footprints:R_0402_1005Metric; symbol jetson-nano-baseboard:R_2k_0402 -> antmicroResistors0402:R_2k_0402
- R75: footprint jetson-nano-baseboard-footprints:R_0402_1005Metric -> antmicro-footprints:R_0402_1005Metric; symbol jetson-nano-baseboard:R_316k_0402 -> antmicroResistors0402:R_316k_0402
- R77: footprint jetson-nano-baseboard-footprints:R_0402_1005Metric -> antmicro-footprints:R_0402_1005Metric; symbol jetson-nano-baseboard:R_60k4_0402 -> antmicroResistors0402:R_60k4_0402
- R84, R86: footprint jetson-nano-baseboard-footprints:R_0402_1005Metric -> antmicro-footprints:R_0402_1005Metric; symbol jetson-nano-baseboard:R_200k_0402 -> antmicroResistors0402:R_200k_0402
- R85: footprint jetson-nano-baseboard-footprints:R_0402_1005Metric -> antmicro-footprints:R_0402_1005Metric; symbol jetson-nano-baseboard:R_470k_0402 -> antmicroResistors0402:R_470k_0402
- R89: footprint jetson-nano-baseboard-footprints:R_0402_1005Metric -> antmicro-footprints:R_0402_1005Metric; symbol jetson-nano-baseboard:R_3R3_0402 -> antmicroResistors0402:R_3R3_0402
- R90: footprint jetson-nano-baseboard-footprints:R_0402_1005Metric -> antmicro-footprints:R_0402_1005Metric; symbol jetson-nano-baseboard:R_26k7_0402 -> antmicroResistors0402:R_26k7_0402
- R94: footprint jetson-nano-baseboard-footprints:R_0402_1005Metric -> antmicro-footprints:R_0402_1005Metric; symbol jetson-nano-baseboard:R_8k66_0402 -> antmicroResistors0402:R_8k66_0402
- T3: footprint jetson-nano-baseboard-footprints:SC70-3 -> antmicro-footprints:SC70-3; symbol jetson-nano-baseboard:BSS138PW -> antmicroTransistorsFETsMOSFETsSingle:BSS138PW
- TP11, TP12, TP15, TP16, TP17, TP40, TP41, TP42, TP44, TP47, TP5, TP8: footprint jetson-nano-baseboard-footprints:TP_SMD_1.5mm -> antmicro-footprints:TP_SMD_1.5mm; symbol jetson-nano-baseboard:TP_1.5mm_SMD -> antmicroTestPoints:TP_1.5mm_SMD
- U1, U5: footprint jetson-nano-baseboard-footprints:SOT-23-5 -> antmicro-footprints:SOT-23-5; symbol jetson-nano-baseboard:LM3671MF-3.3_SOT -> antmicroPMICVoltageRegulatorsDCDCSwitchingRegulators:LM3671MF-3.3_SOT
- U2: footprint jetson-nano-baseboard-footprints:VQFN-HR-14_3.5x4mm -> antmicro-footprints:VQFN-HR-14_3.5x4mm; symbol jetson-nano-baseboard:LM62440-Q1 -> antmicroDCDCConverters:LM62440-Q1
- U3: footprint jetson-nano-baseboard-footprints:SOT-23-6 -> antmicro-footprints:SOT-23-6; symbol jetson-nano-baseboard:SN74LXC1T45DBVR -> antmicroLogicTranslatorsLevelShifters:SN74LXC1T45DBVR
- U6: footprint jetson-nano-baseboard-footprints:SIC47XED-T1-GE3 -> antmicro-footprints:SIC47XED-T1-GE3; symbol jetson-nano-baseboard:SIC477ED-T1-GE3 -> antmicroDCDCConverters:SIC477ED-T1-GE3
