File: usb-debug.kicad_sch (KiCad schematic)
At the start: 87 parts, among them IC1 NCP380LSNAJAAT1G, IC15 TPS7A0518PDBVT, IC3 NCP380LSNAJAAT1G, IC7 HD3SS3220, J11 632723300011, T6 BSS138APW, T7 BSS138APW, T9 BSS138APW, U8 74LVC1G07GV

Commit message: Standardize components
Parts:
- C15, C29: footprint jetson-nano-baseboard-footprints:0402-cap -> antmicro-footprints:C_0402_1005Metric; symbol jetson-nano-baseboard:C_47p_0402 -> antmicroCapacitors0402:C_47p_0402; Author (none) -> Antmicro; Dielectric (none) -> C0G; License (none) -> Apache-2.0; MPN C0402C470J5GACTU -> GRM1555C1E470JA01D; Manufacturer KEMET -> Murata
- C30, C33, C48, C50, C53, C54, C72, C90: footprint jetson-nano-baseboard-footprints:0402-cap -> antmicro-footprints:C_0402_1005Metric; symbol jetson-nano-baseboard:C_100n_0402 -> antmicroCapacitors0402:C_100n_0402; Author (none) -> Antmicro; Dielectric (none) -> X5R; License (none) -> Apache-2.0; MPN 0402X104K6R3CT -> GRM155R61H104KE14D; Manufacturer Walsin -> Murata; Voltage (none) -> 50V
- C31: footprint jetson-nano-baseboard-footprints:1206 -> antmicro-footprints:C_1206_3216Metric; symbol jetson-nano-baseboard:C_100u_1206 -> antmicroCapacitorsmisc:C_100u_1206; Author (none) -> Antmicro; License (none) -> Apache-2.0; MPN C1206C107M9PACTU -> TMCMA0J107MTRF; Manufacturer Kemet -> Vishay; Val (none) -> 100u
- C32: footprint jetson-nano-baseboard-footprints:0402-cap -> antmicro-footprints:C_0402_1005Metric; symbol jetson-nano-baseboard:C_10u_0402 -> antmicroCapacitors0402:C_10u_0402; Author (none) -> Antmicro; License (none) -> Apache-2.0; MPN GRM155R60J106ME44D -> CC0402MRX5R5BB106; Manufacturer MURATA -> Yaego
- C34: footprint jetson-nano-baseboard-footprints:0805-cap -> antmicro-footprints:C_0805_2012Metric; symbol jetson-nano-baseboard:C_47u_0805 -> antmicroCapacitorsmisc:C_47u_0805; Author (none) -> Antmicro; License (none) -> Apache-2.0
- C35: footprint jetson-nano-baseboard-footprints:0603-cap -> antmicro-footprints:C_0603_1608Metric; symbol jetson-nano-baseboard:C_10u_0603 -> antmicroCapacitors0603:C_10u_0603; Author (none) -> Antmicro; License (none) -> Apache-2.0
- C62: footprint jetson-nano-baseboard-footprints:0402-cap -> antmicro-footprints:C_0402_1005Metric; symbol jetson-nano-baseboard:C_4u7_0402 -> antmicroCapacitors0402:C_4u7_0402; Author (none) -> Antmicro; License (none) -> Apache-2.0; Manufacturer MURATA -> Murata
- C66: footprint jetson-nano-baseboard-footprints:0402-cap -> antmicro-footprints:C_0402_1005Metric; symbol jetson-nano-baseboard:C_1u_0402 -> antmicroCapacitors0402:C_1u_0402; Author (none) -> Antmicro; License (none) -> Apache-2.0
- C67: footprint jetson-nano-baseboard-footprints:0402-cap -> antmicro-footprints:C_0402_1005Metric; symbol jetson-nano-baseboard:C_2u2_0402 -> antmicroCapacitors0402:C_2u2_0402; Author (none) -> Antmicro; License (none) -> Apache-2.0
- D17: footprint jetson-nano-baseboard-footprints:SOD-323 -> antmicro-footprints:D_SOD-323F; symbol jetson-nano-baseboard:diode -> antmicroDiodesRectifiersSingle:1N4148WS; Author (none) -> Antmicro; License (none) -> Apache-2.0
- D3, D5: footprint jetson-nano-baseboard-footprints:SOT-23s -> antmicro-footprints:SOT-23-3; symbol jetson-nano-baseboard:PESD2USB5UV-TR -> antmicroTVSDiodes:PESD2USB5UV-TR; Author (none) -> Antmicro; License (none) -> Apache-2.0; Manufacturer Nexperia -> Nexperia
- D6, D7, D8: footprint jetson-nano-baseboard-footprints:TPD4E05U06_PASS -> antmicro-footprints:USON-10_2.5x1mm_P0.5mm; symbol jetson-nano-baseboard:TPD4E05U06_PASS -> antmicroTVSDiodes:TPD4E05U06QDQARQ1; Author (none) -> Antmicro; License (none) -> Apache-2.0; MPN TPD4E05U06DQAR -> TPD4E05U06QDQARQ1
- IC1, IC3: footprint jetson-nano-baseboard-footprints:SOT-23-6 -> antmicro-footprints:SOT-23-6; symbol jetson-nano-baseboard:NCP380LSNAJAAT1G -> antmicroPMICPowerDistributionSwitchesLoadDrivers:NCP380LSNAJAAT1G; Author (none) -> Antmicro; License (none) -> Apache-2.0; Manufacturer onsemi -> ON Semiconductor
- IC15: value TPS7A0518PDBVT -> TPS7A0518P_SOT23-5; footprint jetson-nano-baseboard-footprints:SOT-23-5 -> antmicro-footprints:SOT-23-5; symbol jetson-nano-baseboard:TPS7A0518PDBVT -> antmicroPMICVoltageRegulatorsLinear:TPS7A0518P_SOT23-5; Author (none) -> Antmicro; License (none) -> Apache-2.0
- IC5: value ~ -> FT232R_QFN; footprint jetson-nano-baseboard-footprints:QFN-32 -> antmicro-footprints:QFN-32-1EP_5x5mm; symbol jetson-nano-baseboard:FT232RQ -> antmicroInterfaceControllers:FT232R_QFN; Author (none) -> Antmicro; License (none) -> Apache-2.0; MPN FT232RQ -> FT232RQ-REEL
- IC7: value HD3SS3220 -> HD3SS3220RNH; footprint jetson-nano-baseboard-footprints:RNH0030A -> antmicro-footprints:WQFN-30_1EP_4.6x2.6mm_P0.4mm; symbol jetson-nano-baseboard:HD3SS3220 -> antmicroInterfaceControllers:HD3SS3220RNH; Author (none) -> Antmicro; License (none) -> Apache-2.0; Manufacturer Texas Instrumets -> Texas Instruments
- J11: value 632723300011 -> Conn_USB-C_WE_632723300011; footprint jetson-nano-baseboard-footprints:WE_632723300011 -> antmicro-footprints:Conn_USB-C_WE_632723300011; symbol jetson-nano-baseboard:WE_632723300011 -> antmicroUSBDVIHDMIConnectors:Conn_USB-C_WE_632723300011; Author (none) -> Antmicro; License (none) -> Apache-2.0; Manufacturer Wurth Elektronik -> Würth Elektronik
- J5, J9: value ~ -> USB-Micro-B_0473460001; footprint jetson-nano-baseboard-footprints:CON-Molex-047346-0001 -> antmicro-footprints:USB_Micro_B_Female_0473460001; symbol jetson-nano-baseboard:Micro_USB_B -> antmicroUSBDVIHDMIConnectors:USB-Micro-B_0473460001; Author (none) -> Antmicro; License (none) -> Apache-2.0; MPN 473460001 -> 0473460001; PartSymbol 47346-0001 -> (none)
- L11, L2, L3, L7: value BLM18SG121TN1D -> FB_120Z_3A_0603; footprint jetson-nano-baseboard-footprints:0603 -> antmicro-footprints:FB_0603_1608Metric; symbol jetson-nano-baseboard:BLM18SG121TN1D -> antmicroFerriteBeadsandChips:FB_120Z_3A_0603; Author (none) -> Antmicro; License (none) -> Apache-2.0
- LED1, LED2: footprint jetson-nano-baseboard-footprints:LED0603 -> antmicro-footprints:LED_0603_1608Metric_G; symbol jetson-nano-baseboard:LED -> antmicroLEDIndicationDiscrete:LED_G_0603_LG_L29K-G2J1-24-Z; Author (none) -> Antmicro; License (none) -> Apache-2.0; MPN KPT-1608SGC -> LG L29K-G2J1-24-Z; Manufacturer Kingbright -> Osram
- R102, R47: footprint jetson-nano-baseboard-footprints:0402-res -> antmicro-footprints:R_0402_1005Metric; symbol jetson-nano-baseboard:R_100k_0402 -> antmicroResistors0402:R_100k_0402; Author (none) -> Antmicro; License (none) -> Apache-2.0; MPN CRCW0402100KFKEDHP -> CR0402-FX-1003GLF; Manufacturer VISHAY -> Bourns; Tolerance (none) -> 1%
- R103, R104, R105, R106, R107, R108, R109, R110, R124, R125, R126, R127, R129, R136, R42, R49, R56, R62, R63, R64, R65, R66, R68: footprint jetson-nano-baseboard-footprints:0402-res -> antmicro-footprints:R_0402_1005Metric; symbol jetson-nano-baseboard:R_0R_0402 -> antmicroResistors0402:R_0R_0402; Author (none) -> Antmicro; Current (none) -> 1A; License (none) -> Apache-2.0; Manufacturer PANASONIC -> Panasonic
- R131, R133, R134, R137, R138, R50, R54, R72: footprint jetson-nano-baseboard-footprints:0402-res -> antmicro-footprints:R_0402_1005Metric; symbol jetson-nano-baseboard:R_10k_0402 -> antmicroResistors0402:R_10k_0402; Author (none) -> Antmicro; License (none) -> Apache-2.0; MPN CRCW040210K0FKEDHP -> CR0402-FX-1002GLF; Manufacturer VISHAY -> Bourns; Tolerance (none) -> 1%
- R135, R43: footprint jetson-nano-baseboard-footprints:0402-res -> antmicro-footprints:R_0402_1005Metric; symbol jetson-nano-baseboard:R_470R_0402 -> antmicroResistors0402:R_470R_0402; Author (none) -> Antmicro; License (none) -> Apache-2.0; MPN CRCW0402470RFKED -> CR0402-FX-4700GLF; Manufacturer VISHAY -> Bourns; Tolerance (none) -> 1%
- R20, R41: footprint jetson-nano-baseboard-footprints:0402-res -> antmicro-footprints:R_0402_1005Metric; symbol jetson-nano-baseboard:R_22R_0402 -> antmicroResistors0402:R_22R_0402; Author (none) -> Antmicro; License (none) -> Apache-2.0; MPN CRCW040222R0FKED -> CR0402-FX-22R0GLF; Manufacturer VISHAY -> Bourns; Tolerance (none) -> 1%
- R51: footprint jetson-nano-baseboard-footprints:0402-res -> antmicro-footprints:R_0402_1005Metric; symbol jetson-nano-baseboard:R_909k_0402 -> antmicroResistors0402:R_909k_0402; Author (none) -> Antmicro; License (none) -> Apache-2.0; MPN ERJ2RKF9093X -> CR0402-FX-9093GLF; Manufacturer PANASONIC_ELECTRONIC_COMPONENTS -> Bourns; Tolerance (none) -> 1%
- R53, R67: footprint jetson-nano-baseboard-footprints:0402-res -> antmicro-footprints:R_0402_1005Metric; symbol jetson-nano-baseboard:R_200k_0402 -> antmicroResistors0402:R_200k_0402; Author (none) -> Antmicro; License (none) -> Apache-2.0; MPN RC0402FR-07200KL -> CR0402-FX-2003GLF; Manufacturer YAGEO_(PHYCOMP) -> Bourns; Tolerance (none) -> 1%
- R55, R73: footprint jetson-nano-baseboard-footprints:0402-res -> antmicro-footprints:R_0402_1005Metric; symbol jetson-nano-baseboard:R_2k_0402 -> antmicroResistors0402:R_2k_0402; Author (none) -> Antmicro; License (none) -> Apache-2.0; MPN CRCW04022K00FKED -> CR0402-FX-2001GLF; Manufacturer VISHAY -> Bourns; Tolerance (none) -> 1%
- T6, T7, T9: value BSS138APW -> BSS138PW; footprint jetson-nano-baseboard-footprints:SC70-3 -> antmicro-footprints:SC70-3; symbol jetson-nano-baseboard:BSS138APW -> antmicroTransistorsFETsMOSFETsSingle:BSS138PW; Author (none) -> Antmicro; License (none) -> Apache-2.0; Manufacturer ON Semiconductor -> Nexperia
- TP18, TP19, TP21, TP32: value ~ -> TP_1.5mm_SMD; footprint jetson-nano-baseboard-footprints:TP-R-1.5 -> antmicro-footprints:TP_SMD_1.5mm; symbol jetson-nano-baseboard:Testpad -> antmicroTestPoints:TP_1.5mm_SMD; Author (none) -> Antmicro; License (none) -> Apache-2.0
- U8: value 74LVC1G07GV -> 74LVC1G07_SOT-753; footprint jetson-nano-baseboard-footprints:SOT-753 -> antmicro-footprints:SOT-753; symbol jetson-nano-baseboard:74LVC1G07GV -> antmicroLogicBuffersDriversReceiversTransceivers:74LVC1G07_SOT-753; Author (none) -> Antmicro; License (none) -> Apache-2.0; Manufacturer Texas Instruments -> Nexperia
Connections:
- net 1V8_DBG: now also C66.1; no longer C66.2
- net 3V3_SYS: now also R53.1; no longer R53.2
- net 5V0_DBG: now also C67.1, C72.1, D17.K, L3.1; no longer C67.2, C72.2, D17.C, L3.2 (P)
- net 5V0_SYS: now also C34.1, C90.1, R102.1, R126.1, R134.1, R135.1, R43.1, R47.1, R67.1; no longer C34.2, C90.2, R102.2, R126.2, R134.2, R135.2, R43.2, R47.2, R67.2
- net CC1: now also R66.1; no longer R66.2
- net CC2: now also R65.1; no longer R65.2
- net C_CC2: now also R65.2, R66.2; no longer R65.1, R66.1
- net C_USBSS_RX1_N: now also D6.10
- net C_USBSS_RX1_P: now also D6.9
- net C_USBSS_RX2_N: now also D7.6
- net C_USBSS_RX2_P: now also D7.7
- net C_USBSS_TX1_N: now also C50.2, D6.6; no longer C50.1
- net C_USBSS_TX1_P: now also C48.2, D6.7; no longer C48.1
- net C_USBSS_TX2_N: now also C54.2, D7.10; no longer C54.1
- net C_USBSS_TX2_P: now also C53.2, D7.9; no longer C53.1
- net DBG_USB_D_N: now also C29.1; no longer C29.2
- net DBG_USB_D_P: now also C15.1; no longer C15.2
- net GND: now also C15.2, C29.2, C30.2, C31.2, C34.2, C35.2, C62.2, C66.2, C67.2, C72.2, C90.2, IC5.33 (EP), J11.SH, J9.SH (SHIELD), L7.2, R127.2, R131.2, R137.2; no longer C15.1, C29.1, C30.1, C31.1, C34.1, C35.1, C62.1, C66.1, C67.1, C72.1, C90.1, J11.Shell (Shield), J9.S (SHIELD), L7.1 (P), R127.1, R131.1, R137.1
- net OTG_USB_D_N: now also D8.10
- net OTG_USB_D_P: now also D8.9
- net OTG_USB_ID: now also D8.7, R134.2; no longer R134.1
- net OTG_USB_VBUS: now also C62.1, R72.2; no longer C62.2, R72.1
- net UART1_RX: now also R20.1; no longer R20.2
- net UART1_TX: now also R41.1; no longer R41.2
- net USBC_ADDR: now also R126.2, R127.1; no longer R126.1, R127.2
- net USBC_ID: now also R47.2; no longer R47.1
- net USBC_INTN: now also R67.2; no longer R67.1
- net USBC_VBUS: now also C35.1, R131.1; no longer C35.2, R131.2
- net USBSS_TX1_N: now also C48.1, IC7.16 (TX1-); no longer C50.2, IC7.17 (TX1p)
- net USBSS_TX1_P: now also C50.1, IC7.17 (TX1+); no longer C48.2, IC7.16 (TX1n)
- net USBSS_TX2_N: now also C53.1, IC7.20 (TX2-); no longer C54.2, IC7.21 (TX2p)
- net USBSS_TX2_P: now also C54.1, IC7.21 (TX2+); no longer C53.2, IC7.20 (TX2n)
- net USB_DBG_VBUS: now also L3.2; no longer L3.1 (P)
- net ~{OTG_USB_VBUS_DET}: now also R129.1; no longer R129.2
- net at IC3.6 (OUT), L2.1, R42.2: now also C31.1; no longer C31.2
- net at IC5.16 (3V3OUT): now also C30.1; no longer C30.2
- net at IC5.2 (RXD): now also R41.2; no longer R41.1
- net at IC5.30 (TXD): now also R20.2; no longer R20.1
- net at IC7.11 (DIR): now also R53.2; no longer R53.1
- net at LED1.1: now also R43.2; no longer R43.1
- net at R73.1, T6.1 (G): now also R72.1; no longer R72.2
- net at T6.3 (D), T9.2 (S): now also R129.2; no longer R129.1
- net at IC3.3 (~{EN}), R49.2, T7.3 (D): now also R102.2, R137.1; no longer R102.1, R137.2
- net at LED2.1: now also R135.2; no longer R135.1
- net at D8.5: now also D8.6
- new net: J5.SH (SHIELD), L7.1
Other:
- moved on the sheet: C15, C29, C30, C32, C33, C34, C35, C48, C50, C53, C54, C62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

Commit message: [#56834] Fix components links
Parts:
- C15, C29: footprint antmicro-footprints:C_0402_1005Metric -> jetson-nano-baseboard-footprints:C_0402_1005Metric; symbol antmicroCapacitors0402:C_47p_0402 -> jetson-nano-baseboard:C_47p_0402; MPN GRM1555C1E470JA01D -> C0402C470J5GACTU; Manufacturer Murata -> KEMET
- C30, C33, C48, C50, C53, C54, C72, C90: footprint antmicro-footprints:C_0402_1005Metric -> jetson-nano-baseboard-footprints:C_0402_1005Metric; symbol antmicroCapacitors0402:C_100n_0402 -> jetson-nano-baseboard:C_100n_0402
- C31: value 100u -> C_100u_1206; footprint antmicro-footprints:C_1206_3216Metric -> jetson-nano-baseboard-footprints:C_1206_3216Metric; symbol antmicroCapacitorsmisc:C_100u_1206 -> jetson-nano-baseboard:C_100u_1206; MPN TMCMA0J107MTRF -> GRM31CR60J107MEA8K; Manufacturer Vishay -> Murata; Voltage 6.3V -> (none)
- C32: footprint antmicro-footprints:C_0402_1005Metric -> jetson-nano-baseboard-footprints:C_0402_1005Metric; symbol antmicroCapacitors0402:C_10u_0402 -> jetson-nano-baseboard:C_10u_0402; Manufacturer Yaego -> YAGEO
- C34: footprint antmicro-footprints:C_0805_2012Metric -> jetson-nano-baseboard-footprints:C_0805_2012Metric; symbol antmicroCapacitorsmisc:C_47u_0805 -> jetson-nano-baseboard:C_47u_0805
- C35: footprint antmicro-footprints:C_0603_1608Metric -> jetson-nano-baseboard-footprints:C_0603_1608Metric; symbol antmicroCapacitors0603:C_10u_0603 -> jetson-nano-baseboard:C_10u_0603
- C62: footprint antmicro-footprints:C_0402_1005Metric -> jetson-nano-baseboard-footprints:C_0402_1005Metric; symbol antmicroCapacitors0402:C_4u7_0402 -> jetson-nano-baseboard:C_4u7_0402
- C66: footprint antmicro-footprints:C_0402_1005Metric -> jetson-nano-baseboard-footprints:C_0402_1005Metric; symbol antmicroCapacitors0402:C_1u_0402 -> jetson-nano-baseboard:C_1u_0402
- C67: footprint antmicro-footprints:C_0402_1005Metric -> jetson-nano-baseboard-footprints:C_0402_1005Metric; symbol antmicroCapacitors0402:C_2u2_0402 -> jetson-nano-baseboard:C_2u2_0402
- D17: footprint antmicro-footprints:D_SOD-323F -> jetson-nano-baseboard-footprints:D_SOD-323F; symbol antmicroDiodesRectifiersSingle:1N4148WS -> jetson-nano-baseboard:1N4148WS
- D3, D5: footprint antmicro-footprints:SOT-23-3 -> jetson-nano-baseboard-footprints:SOT-23-3; symbol antmicroTVSDiodes:PESD2USB5UV-TR -> jetson-nano-baseboard:PESD2USB5UV-TR; MPN PESD2USB5UV-TR -> PESD2USB5UV-TR
- D6, D7, D8: value TPD4E05U06_PASS -> TPD4E05U06QDQARQ1; footprint antmicro-footprints:USON-10_2.5x1mm_P0.5mm -> jetson-nano-baseboard-footprints:USON-10_2.5x1mm_P0.5mm; symbol antmicroTVSDiodes:TPD4E05U06QDQARQ1 -> jetson-nano-baseboard:TPD4E05U06QDQARQ1
- IC1, IC3: footprint antmicro-footprints:SOT-23-6 -> jetson-nano-baseboard-footprints:SOT-23-6; symbol antmicroPMICPowerDistributionSwitchesLoadDrivers:NCP380LSNAJAAT1G -> jetson-nano-baseboard:NCP380LSNAJAAT1G
- IC15: footprint antmicro-footprints:SOT-23-5 -> jetson-nano-baseboard-footprints:SOT-23-5; symbol antmicroPMICVoltageRegulatorsLinear:TPS7A0518P_SOT23-5 -> jetson-nano-baseboard:TPS7A0518P_SOT23-5
- IC5: footprint antmicro-footprints:QFN-32-1EP_5x5mm -> jetson-nano-baseboard-footprints:QFN-32-1EP_5x5mm; symbol antmicroInterfaceControllers:FT232R_QFN -> jetson-nano-baseboard:FT232R_QFN; Manufacturer FTDI -> FTDI Chip
- IC7: footprint antmicro-footprints:WQFN-30_1EP_4.6x2.6mm_P0.4mm -> jetson-nano-baseboard-footprints:WQFN-30-1EP_4.6x2.6mm_P0.4mm; symbol antmicroInterfaceControllers:HD3SS3220RNH -> jetson-nano-baseboard:HD3SS3220RNH
- J11: value Conn_USB-C_WE_632723300011 -> USB-C_WE_632723300011; footprint antmicro-footprints:Conn_USB-C_WE_632723300011 -> jetson-nano-baseboard-footprints:USB-C_Receptacle_WE_632723300011; symbol antmicroUSBDVIHDMIConnectors:Conn_USB-C_WE_632723300011 -> jetson-nano-baseboard:USB-C_WE_632723300011
- J5, J9: value USB-Micro-B_0473460001 -> USB-Micro-B_Molex_473460001; footprint antmicro-footprints:USB_Micro_B_Female_0473460001 -> jetson-nano-baseboard-footprints:USB-Micro-B_Receptacle_Molex_473460001; symbol antmicroUSBDVIHDMIConnectors:USB-Micro-B_0473460001 -> jetson-nano-baseboard:USB-Micro-B_Molex_473460001; MPN 0473460001 -> 473460001
- L11, L2, L3, L7: value FB_120Z_3A_0603 -> FB_120Z_3A_Murata-BLM18SG_0603; footprint antmicro-footprints:FB_0603_1608Metric -> jetson-nano-baseboard-footprints:FB_0603_1608Metric; symbol antmicroFerriteBeadsandChips:FB_120Z_3A_0603 -> jetson-nano-baseboard:FB_120Z_3A_Murata-BLM18SG_0603
- LED1, LED2: value ~ -> LED_G_0603_LG_L29K-G2J1-24-Z; footprint antmicro-footprints:LED_0603_1608Metric_G -> jetson-nano-baseboard-footprints:LED_0603_1608Metric_G; symbol antmicroLEDIndicationDiscrete:LED_G_0603_LG_L29K-G2J1-24-Z -> jetson-nano-baseboard:LED_G_0603_LG_L29K-G2J1-24-Z; Manufacturer Osram -> OSRAM
- R102, R47: footprint antmicro-footprints:R_0402_1005Metric -> jetson-nano-baseboard-footprints:R_0402_1005Metric; symbol antmicroResistors0402:R_100k_0402 -> jetson-nano-baseboard:R_100k_0402
- R103, R104, R105, R106, R107, R108, R109, R110, R49, R56, R62, R63, R65: footprint antmicro-footprints:R_0402_1005Metric -> jetson-nano-baseboard-footprints:R_0402_1005Metric; symbol antmicroResistors0402:R_0R_0402 -> jetson-nano-baseboard:R_0R_0402
- R124, R125, R126, R127, R129, R136, R42, R64, R66, R68: footprint antmicro-footprints:R_0402_1005Metric -> jetson-nano-baseboard-footprints:R_0402_1005Metric; symbol antmicroResistors0402:R_0R_0402 -> jetson-nano-baseboard:R_0R_0402; now not fitted; now left out of the parts list
- R131, R133, R134, R138, R50, R72: footprint antmicro-footprints:R_0402_1005Metric -> jetson-nano-baseboard-footprints:R_0402_1005Metric; symbol antmicroResistors0402:R_10k_0402 -> jetson-nano-baseboard:R_10k_0402
- R135, R43: footprint antmicro-footprints:R_0402_1005Metric -> jetson-nano-baseboard-footprints:R_0402_1005Metric; symbol antmicroResistors0402:R_470R_0402 -> jetson-nano-baseboard:R_470R_0402
- R137, R54: footprint antmicro-footprints:R_0402_1005Metric -> jetson-nano-baseboard-footprints:R_0402_1005Metric; symbol antmicroResistors0402:R_10k_0402 -> jetson-nano-baseboard:R_10k_0402; now not fitted; now left out of the parts list
- R20, R41: footprint antmicro-footprints:R_0402_1005Metric -> jetson-nano-baseboard-footprints:R_0402_1005Metric; symbol antmicroResistors0402:R_22R_0402 -> jetson-nano-baseboard:R_22R_0402
- R51: footprint antmicro-footprints:R_0402_1005Metric -> jetson-nano-baseboard-footprints:R_0402_1005Metric; symbol antmicroResistors0402:R_909k_0402 -> jetson-nano-baseboard:R_909k_0402
- R53, R67: footprint antmicro-footprints:R_0402_1005Metric -> jetson-nano-baseboard-footprints:R_0402_1005Metric; symbol antmicroResistors0402:R_200k_0402 -> jetson-nano-baseboard:R_200k_0402
- R55, R73: footprint antmicro-footprints:R_0402_1005Metric -> jetson-nano-baseboard-footprints:R_0402_1005Metric; symbol antmicroResistors0402:R_2k_0402 -> jetson-nano-baseboard:R_2k_0402
- T6, T9: footprint antmicro-footprints:SC70-3 -> jetson-nano-baseboard-footprints:SC70-3; symbol antmicroTransistorsFETsMOSFETsSingle:BSS138PW -> jetson-nano-baseboard:BSS138PW
- T7: footprint antmicro-footprints:SC70-3 -> jetson-nano-baseboard-footprints:SC70-3; symbol antmicroTransistorsFETsMOSFETsSingle:BSS138PW -> jetson-nano-baseboard:BSS138PW; now not fitted; now left out of the parts list
- TP18, TP19, TP21, TP32: footprint antmicro-footprints:TP_SMD_1.5mm -> jetson-nano-baseboard-footprints:TP_SMD_1.5mm; symbol antmicroTestPoints:TP_1.5mm_SMD -> jetson-nano-baseboard:TP_1.5mm_SMD; MPN N/A -> (none); Manufacturer N/A -> (none)
- U8: footprint antmicro-footprints:SOT-753 -> jetson-nano-baseboard-footprints:SOT-753; symbol antmicroLogicBuffersDriversReceiversTransceivers:74LVC1G07_SOT-753 -> jetson-nano-baseboard:74LVC1G07_SOT-753

Commit message: [#57913] fix 2309413-1
Parts:
- C15, C29: footprint jetson-nano-baseboard-footprints:C_0402_1005Metric -> antmicro-footprints:C_0402_1005Metric; symbol jetson-nano-baseboard:C_47p_0402 -> antmicroCapacitors0402:C_47p_0402
- C30, C33, C48, C50, C53, C54, C72, C90: footprint jetson-nano-baseboard-footprints:C_0402_1005Metric -> antmicro-footprints:C_0402_1005Metric; symbol jetson-nano-baseboard:C_100n_0402 -> antmicroCapacitors0402:C_100n_0402
- C31: footprint jetson-nano-baseboard-footprints:C_1206_3216Metric -> antmicro-footprints:C_1206_3216Metric; symbol jetson-nano-baseboard:C_100u_1206 -> antmicroCapacitorsmisc:C_100u_1206
- C32: footprint jetson-nano-baseboard-footprints:C_0402_1005Metric -> antmicro-footprints:C_0402_1005Metric; symbol jetson-nano-baseboard:C_10u_0402 -> antmicroCapacitors0402:C_10u_0402
- C34: footprint jetson-nano-baseboard-footprints:C_0805_2012Metric -> antmicro-footprints:C_0805_2012Metric; symbol jetson-nano-baseboard:C_47u_0805 -> antmicroCapacitorsmisc:C_47u_0805
- C35: footprint jetson-nano-baseboard-footprints:C_0603_1608Metric -> antmicro-footprints:C_0603_1608Metric; symbol jetson-nano-baseboard:C_10u_0603 -> antmicroCapacitors0603:C_10u_0603
- C62: footprint jetson-nano-baseboard-footprints:C_0402_1005Metric -> antmicro-footprints:C_0402_1005Metric; symbol jetson-nano-baseboard:C_4u7_0402 -> antmicroCapacitors0402:C_4u7_0402
- C66: footprint jetson-nano-baseboard-footprints:C_0402_1005Metric -> antmicro-footprints:C_0402_1005Metric; symbol jetson-nano-baseboard:C_1u_0402 -> antmicroCapacitors0402:C_1u_0402
- C67: footprint jetson-nano-baseboard-footprints:C_0402_1005Metric -> antmicro-footprints:C_0402_1005Metric; symbol jetson-nano-baseboard:C_2u2_0402 -> antmicroCapacitors0402:C_2u2_0402
- D17: footprint jetson-nano-baseboard-footprints:D_SOD-323F -> antmicro-footprints:D_SOD-323F; symbol jetson-nano-baseboard:1N4148WS -> antmicroDiodesRectifiersSingle:1N4148WS
- D3, D5: footprint jetson-nano-baseboard-footprints:SOT-23-3 -> antmicro-footprints:SOT-23-3; symbol jetson-nano-baseboard:PESD2USB5UV-TR -> antmicroTVSDiodes:PESD2USB5UV-TR
- D6, D7, D8: footprint jetson-nano-baseboard-footprints:USON-10_2.5x1mm_P0.5mm -> antmicro-footprints:USON-10_2.5x1mm_P0.5mm; symbol jetson-nano-baseboard:TPD4E05U06QDQARQ1 -> antmicroTVSDiodes:TPD4E05U06QDQARQ1
- IC1, IC3: footprint jetson-nano-baseboard-footprints:SOT-23-6 -> antmicro-footprints:SOT-23-6; symbol jetson-nano-baseboard:NCP380LSNAJAAT1G -> antmicroPMICPowerDistributionSwitchesLoadDrivers:NCP380LSNAJAAT1G
- IC15: footprint jetson-nano-baseboard-footprints:SOT-23-5 -> antmicro-footprints:SOT-23-5; symbol jetson-nano-baseboard:TPS7A0518P_SOT23-5 -> antmicroPMICVoltageRegulatorsLinear:TPS7A0518P_SOT23-5
- IC5: footprint jetson-nano-baseboard-footprints:QFN-32-1EP_5x5mm -> antmicro-footprints:QFN-32-1EP_5x5mm; symbol jetson-nano-baseboard:FT232R_QFN -> antmicroInterfaceControllers:FT232R_QFN
- IC7: footprint jetson-nano-baseboard-footprints:WQFN-30-1EP_4.6x2.6mm_P0.4mm -> antmicro-footprints:WQFN-30-1EP_4.6x2.6mm_P0.4mm; symbol jetson-nano-baseboard:HD3SS3220RNH -> antmicroInterfaceControllers:HD3SS3220RNH
- J11: footprint jetson-nano-baseboard-footprints:USB-C_Receptacle_WE_632723300011 -> antmicro-footprints:USB-C_Receptacle_WE_632723300011; symbol jetson-nano-baseboard:USB-C_WE_632723300011 -> antmicroUSBConnectors:USB-C_WE_632723300011
- J5, J9: footprint jetson-nano-baseboard-footprints:USB-Micro-B_Receptacle_Molex_473460001 -> antmicro-footprints:USB-Micro-B_Receptacle_Molex_473460001; symbol jetson-nano-baseboard:USB-Micro-B_Molex_473460001 -> antmicroUSBConnectors:USB-Micro-B_Molex_473460001
- L11, L2, L3, L7: footprint jetson-nano-baseboard-footprints:FB_0603_1608Metric -> antmicro-footprints:FB_0603_1608Metric; symbol jetson-nano-baseboard:FB_120Z_3A_Murata-BLM18SG_0603 -> antmicroFerriteBeadsandChips:FB_120Z_3A_Murata-BLM18SG_0603
- LED1, LED2: footprint jetson-nano-baseboard-footprints:LED_0603_1608Metric_G -> antmicro-footprints:LED_0603_1608Metric_G; symbol jetson-nano-baseboard:LED_G_0603_LG_L29K-G2J1-24-Z -> antmicroLEDIndicationDiscrete:LED_G_0603_LG_L29K-G2J1-24-Z
- R102, R47: footprint jetson-nano-baseboard-footprints:R_0402_1005Metric -> antmicro-footprints:R_0402_1005Metric; symbol jetson-nano-baseboard:R_100k_0402 -> antmicroResistors0402:R_100k_0402
- R103, R104, R105, R106, R107, R108, R109, R110, R124, R125, R126, R127, R129, R136, R42, R49, R56, R62, R63, R64, R65, R66, R68: footprint jetson-nano-baseboard-footprints:R_0402_1005Metric -> antmicro-footprints:R_0402_1005Metric; symbol jetson-nano-baseboard:R_0R_0402 -> antmicroResistors0402:R_0R_0402
- R131, R133, R134, R137, R138, R50, R54, R72: footprint jetson-nano-baseboard-footprints:R_0402_1005Metric -> antmicro-footprints:R_0402_1005Metric; symbol jetson-nano-baseboard:R_10k_0402 -> antmicroResistors0402:R_10k_0402
- R135, R43: footprint jetson-nano-baseboard-footprints:R_0402_1005Metric -> antmicro-footprints:R_0402_1005Metric; symbol jetson-nano-baseboard:R_470R_0402 -> antmicroResistors0402:R_470R_0402
- R20, R41: footprint jetson-nano-baseboard-footprints:R_0402_1005Metric -> antmicro-footprints:R_0402_1005Metric; symbol jetson-nano-baseboard:R_22R_0402 -> antmicroResistors0402:R_22R_0402
- R51: footprint jetson-nano-baseboard-footprints:R_0402_1005Metric -> antmicro-footprints:R_0402_1005Metric; symbol jetson-nano-baseboard:R_909k_0402 -> antmicroResistors0402:R_909k_0402
- R53, R67: footprint jetson-nano-baseboard-footprints:R_0402_1005Metric -> antmicro-footprints:R_0402_1005Metric; symbol jetson-nano-baseboard:R_200k_0402 -> antmicroResistors0402:R_200k_0402
- R55, R73: footprint jetson-nano-baseboard-footprints:R_0402_1005Metric -> antmicro-footprints:R_0402_1005Metric; symbol jetson-nano-baseboard:R_2k_0402 -> antmicroResistors0402:R_2k_0402
- T6, T7, T9: footprint jetson-nano-baseboard-footprints:SC70-3 -> antmicro-footprints:SC70-3; symbol jetson-nano-baseboard:BSS138PW -> antmicroTransistorsFETsMOSFETsSingle:BSS138PW
- TP18, TP19, TP21, TP32: footprint jetson-nano-baseboard-footprints:TP_SMD_1.5mm -> antmicro-footprints:TP_SMD_1.5mm; symbol jetson-nano-baseboard:TP_1.5mm_SMD -> antmicroTestPoints:TP_1.5mm_SMD
- U8: footprint jetson-nano-baseboard-footprints:SOT-753 -> antmicro-footprints:SOT-753; symbol jetson-nano-baseboard:74LVC1G07_SOT-753 -> antmicroLogicBuffersDriversReceiversTransceivers:74LVC1G07_SOT-753

Commit message: [#83358] Update KiCad project files
Connections:
- net 5V0_DBG: no longer D17.K
- net 5V0_SYS: now also D17.1 (C); no longer D17.A
- net DBG_USB_D_N: now also J9.3 (D+); no longer J9.2 (D-)
- net DBG_USB_D_P: no longer J9.3 (D+)
- net GND: no longer J5.5 (GND), J9.5 (GND), J9.SH (SHIELD)
- net OTG_USB_D_N: now also J5.3 (D+); no longer J5.2 (D-)
- net OTG_USB_D_P: no longer J5.3 (D+)
- net OTG_USB_ID: now also J5.2 (D-); no longer J5.4 (ID)
- net USB1_D_N: no longer J11.A7 (D-)
- net USB1_D_P: no longer J11.A6 (D+)
- net ~{OTG_USB_FAULT}: no longer LED2.2
- net at L7.1: no longer J5.SH (SHIELD)
- net at LED1.2 (A): no longer IC3.4 (~{FAULT})
